File: kicad/CPU6.kicad_sch (KiCad schematic)
At the start: 117 parts

Commit message: All chips on schematic
Parts:
- removed UA13, UM10: (no value), symbol 74xx:74LS37
- removed UA14, UA2, UA3: (no value), symbol 74xx:74LS38
- removed UK9: (no value), symbol 74xx:74LS151
- added P3: Connector, symbol Connector_Generic:Conn_02x13_Top_Bottom
- added R12: 1k0, symbol Device:R
- added R13, R14, R9, R? (x2): (no value), symbol Device:R
- added U?: (no value), symbol 74xx:74LS157
- added U?, UM14: (no value), symbol 74xx:74LS240
- added UA13, UM10: (no value), symbol oldchips:7437
- added UA14, UA2: (no value), symbol oldchips:7438
- added UB12, UD12, UL14: (no value), symbol 74xx:74LS00
- added UC10: (no value), symbol 74xx:74LS04
- added UD10: (no value), symbol 74xx:74LS02
- added UD7: (no value), symbol oldchips:74120
- added UD8: (no value), symbol 74xx:74LS20
- added UK9: (no value), symbol oldchips:74S151
- added UL13: (no value), symbol 74xx:74LS109
- added UM12: (no value), symbol 74xx:74LS378
- added UM13: (no value), symbol 74xx:74LS259
- gave numbers to parts that had none: 2
- renumbered UE12 to UE10, UE13 to UE12
Connections:
- net MC24 is gone; now on net K12.8: UJ5.19 (Q7)
- net MC25 is gone; now on net H13.12: UJ5.16 (Q6)
- net (WK.CLK): no longer UD6.9 (Zc)
- net A12: now also UC7.6
- net A15: now also UC8.3
- net A8: now also UC8.9
- net DB0: now also J?.b21 (Pin_b21); no longer J?.a21 (Pin_a21)
- net DB1: now also J?.b22 (Pin_b22); no longer J?.a22 (Pin_a22)
- net DB2: now also J?.b23 (Pin_b23); no longer J?.a23 (Pin_a23)
- net DB3: now also J?.b24 (Pin_b24); no longer J?.a24 (Pin_a24)
- net DB4: now also J?.b25 (Pin_b25); no longer J?.a25 (Pin_a25)
- net DB5: now also J?.b26 (Pin_b26); no longer J?.a26 (Pin_a26)
- net DB6: now also J?.b27 (Pin_b27); no longer J?.a27 (Pin_a27)
- net DB7: now also J?.b28 (Pin_b28); no longer J?.a28 (Pin_a28)
- net DP0: now also UH14.9 (O4a)
- net DP?: now also UC11.6 (Q3)
- net F5: now also UC9.14 (D5)
- net M12.10: now also UK13.6 (I0a); no longer UK10.10
- net MC0: now also UJ12.14 (S0), UK9.11 (S0)
- net MC1: now also UJ12.2 (S1), UK9.10 (S1)
- net MC2: now also UJ11.7 (~{E}), UK9.9 (S2)
- net MC26: now also UH11.1 (A0)
- net MC27: now also UH11.2 (A1)
- net MC29: now also UE7.1 (A0)
- net MC3: now also UJ11.11 (S0)
- net MC31: now also UK9.7 (~{E})
- net MC4: now also UJ11.10 (S1), UJ13.14 (S0)
- net MC5: now also UJ10.7 (~{E}), UJ13.2 (S1)
- net MC6: now also UJ10.11 (S0), UK13.2 (S1)
- net MC7: now also UJ10.10 (S1), UK10.11, UK13.14 (S0)
- net PA11: now also J?.b16 (Pin_b16); no longer J?.a16 (Pin_a16)
- net PA12: now also J?.b17 (Pin_b17); no longer J?.a17 (Pin_a17), UB8.4, UC8.11
- net PA13: now also J?.b18 (Pin_b18); no longer J?.a18 (Pin_a18), UB8.3, UC7.8
- net PA14: now also J?.b19 (Pin_b19), UA9.12 (BUS2); no longer J?.a19 (Pin_a19), UA8.12 (BUS2)
- net PA15: now also J?.b20 (Pin_b20), UA10.12 (BUS2); no longer J?.a20 (Pin_a20), UA8.1 (BUS0)
- net PA?? (18): now also J?.a18 (Pin_a18); no longer J?.b18 (Pin_b18)
- net PA?? (19): now also J?.a19 (Pin_a19), UA8.12 (BUS2); no longer J?.b19 (Pin_b19), UA10.12 (BUS2)
- net PA?? (20): now also J?.a20 (Pin_a20); no longer J?.b20 (Pin_b20)
- net PA?? (23): now also J?.a23 (Pin_a23); no longer J?.b23 (Pin_b23)
- net PA?? (24): now also J?.a24 (Pin_a24); no longer J?.b24 (Pin_b24)
- net PA?? (25): now also J?.a25 (Pin_a25); no longer J?.b25 (Pin_b25)
- net ~{A13}: now also J?.a12 (Pin_a12); no longer J?.b12 (Pin_b12)
- net ~{A??}: now also J?.a10 (Pin_a10), J?.a9 (Pin_a9); no longer J?.b10 (Pin_b10), J?.b9 (Pin_b9)
- net ~{BUSRESET}: now also UF12.1 (~{R}); no longer UD4.1 (~{Mr})
- net ~{LOAD.RIR}: now also UC13.1 (~{E})
- net ~{PROME}: now also UL6.10
- net ~{READ.ADR.LO}: now also UD4.10 (Q3)
- net ~{READ.ILR}: now also UA8.7 (~{R})
- net at UK12.2: now also UK12.3, UK12.4
- net B15.9: now reaches UD6.1 (S)
- net at UE8.11: now also UD10.5, UD8.12, UD8.2
- net VCC: now reaches UL6.14 (VCC)
- net VCC: now also E15.14 (VCC), RN?.1 (common), RN?.10 (COM2), UA1.14 (VCC), UA15.14 (VCC), UA3.14 (VCC), UB11.14 (VCC), UB15.14 (VCC), UB7.14 (VCC), UB8.14 (VCC), UC7.14 (VCC), UC8.14 (VCC), UD2.16 (VCC), UE10.14 (VCC), UE11.14 (VCC), UE12.14 (VCC), UE14.14 (VCC), UE8.14 (VCC), UF14.14 (VCC), UH13.14 (VCC), UJ6.14 (VCC), UK10.14 (VCC), UK12.14 (VCC), UK6.14 (VCC), UL10.14 (VCC), UM9.14 (VCC), R12.1, R13.1, R14.1, R9.1, UA13.14 (VCC), UA14.14 (VCC), UA2.14 (VCC), UB12.14 (VCC), UC10.14 (VCC), UD10.14 (VCC), UD12.14 (VCC), UD8.14 (VCC), UL13.16 (VCC), UL14.14 (VCC), UM10.14 (VCC)
- net GND: now reaches UL6.7 (GND)
- net GND: now also E15.7 (GND), RN?.1 (COM1), SW?.10, SW?.11, SW?.12, SW?.13, SW?.14, SW?.15, SW?.16, SW?.9, UA1.12 (D), UA1.2 (D), UA1.7 (GND), UA15.7 (GND), UA3.7 (GND), UB1.10 (~{CET}), UB1.8 (GND), UB11.7 (GND), UB15.7 (GND), UB7.7 (GND), UB8.7 (GND), UC7.7 (GND), UC8.7 (GND), UD2.8 (GND), UE10.7 (GND), UE11.7 (GND), UE12.7 (GND), UE14.7 (GND), UE7.3 (A2), UE7.4 (E1), UE7.5 (E2), UE7.8 (GND), UE8.7 (GND), UF14.7 (GND), UH13.7 (GND), UJ6.7 (GND), UK10.7 (GND), UK12.7 (GND), UK6.7 (GND), UL10.7 (GND), UM9.7 (GND), UA13.7 (GND), UA14.7 (GND), UA2.7 (GND), UB12.7 (GND), UC10.7 (GND), UD10.7 (GND), UD12.7 (GND), UD8.7 (GND), UL13.8 (GND), UL14.7 (GND), UM10.7 (GND)
- net ~{READ.SW1}: now reaches UM7.1 (OEa)
- net ~{READ.SW1}: now also UA7.1 (OEa), UD5.5 (Q1)
- net at UM7.11 (I0b): now also RN?.7 (R6), SW?.4
- net at UM7.12 (O3a): now also UM7.9 (O0b)
- net at UM7.13 (I1b): now also RN?.3 (R2), RN?.5 (R4), SW?.3, SW?.7, UM7.6 (I2a)
- net at UM7.15 (I2b): now also RN?.6 (R5), SW?.2
- net L15.11: now reaches UM7.17 (I3b)
- net at UM7.19 (OEb): now also UM14.1 (OEa)
- net F14.1: now reaches RN?.4 (R3), SW?.6, UM7.4 (I1a)
- net B11.5: now reaches UF12.3 (C)
- net D7.7: now reaches UF12.4 (~{S})
- net D7.7: now also UA1.10 (~{S})
- net M10.10: now reaches UF12.5 (Q)
- net M13.6: now reaches UF14.10
- net at UF14.8: now also UF13.14 (D5)
- net M9.9: now reaches UF14.9
- net ~{LOAD.DB}: now reaches UA11.1 (~{RLE}), UA12.1 (~{RLE})
- net ~{LOAD.DB}: now also UE6.7 (O7)
- net ~{READ.DB}: now reaches UA11.11 (~{OE}), UA12.11 (~{OE})
- net ~{READ.DB}: now also UD5.15 (Q5)
- net at UA5.1 (BUS0): now also J?.b9 (Pin_b9); no longer J?.a9 (Pin_a9)
- net at UA5.12 (BUS2): now also J?.b12 (Pin_b12); no longer J?.a12 (Pin_a12)
- net at UA5.15 (BUS3): now also J?.b11 (Pin_b11); no longer J?.a11 (Pin_a11)
- net at UA5.4 (BUS1): now also J?.b10 (Pin_b10); no longer J?.a10 (Pin_a10)
- net at Uf12.11 (C): now also UF13.9 (Cp)
- net E6.12: now reaches UD9.1 (~{E})
- net at UD9.12 (Q4): now also UD10.11
- net at UD9.2 (Q0): now also UA8.14 (IN3)
- net at UD9.5 (Q1): now also UD10.9
- net at UE11.10: now also UE11.9, UE14.11 (C)
- net at UE11.11: now also UE14.9 (Q)
- net at UE11.8: now also UE10.1
- net at YM11.1: now also R?.1, R?.1, UM10.5
- net at YM11.2: now also R?.2, U?.3 (I1a), UM10.6
- net ~{2901.OE}: now reaches UF10.40 (~{OE})
- net ~{2901.OE}: now also UF11.40 (~{OE}), UL6.8
- net at UE12.12: no longer UE12.10
- net at UE12.13: no longer UE12.11
- net at UA15.3: now also UA15.8, UA13.4, UA13.5
- net C15.2: now reaches UA15.4
- net A1.6: now reaches UB11.3
- net F12.3: now reaches UB11.4
- net F12.3: now also UB11.5
- net C15.9: now reaches UB11.6
- net T22: now reaches UC8.2
- net at UM9.10 (~{S}): now also RN?.7 (R6)
- net at UM9.13 (~{R}): now also UM13.10 (Q5)
- net F14.10: now reaches UM9.9 (Q)
- net at UH13.10: now also UH13.9, UK12.10
- net H13.12: now reaches UH13.12
- net H13.12: now also UK11.3 (A2)
- net ~{REG.WE}: now reaches UH13.8
- net ~{REG.WE}: now also UD14.20 (~{WE}), UD15.20 (~{WE})
- net ~{READ.PA}: now reaches UD5.2 (Q0)
- net ~{READ.PA}: now also UA10.7 (~{R}), UA9.7 (~{R})
- net ~{READ.SW2}: now reaches UD5.7 (Q2)
- net at UL10.1 (~{R}), UL10.13 (~{R}): now also R9.2, U?.1 (S)
- net at UL10.2 (D), UL10.9 (Q): now also U?.13 (I1d), UM10.12
- net at UL10.11 (C), UL10.3 (C): now also U?.4 (Za)
- net at UL10.4 (~{S}): now also UL10.10 (~{S})
- net at UL10.6 (~{Q}): now also U?.10 (I1c)
- net at P2.9 (Pin_9): now also UM10.8
- net at UE8.1: now also UE11.1, UE14.2 (D)
- net at UE8.2: now also UE8.4
- net at UA4.1 (BUS0): now also J?.b5 (Pin_b5); no longer J?.a5 (Pin_a5)
- net at UA4.12 (BUS2): now also J?.b8 (Pin_b8); no longer J?.a8 (Pin_a8)
- net at UA4.15 (BUS3): now also J?.b7 (Pin_b7); no longer J?.a7 (Pin_a7)
- net at UA4.4 (BUS1): now also J?.b6 (Pin_b6); no longer J?.a6 (Pin_a6)
- net at UA15.2: now also UA14.10
- net IPA14: now reaches UC7.11
- net K12.9: now reaches UE5.15 (Q5)
- net K12.9: now also UK11.1 (A0), UK12.9
- net M7.4: now reaches UF14.1
- net H14.2: now reaches UF14.2
- net H14.2: now also UE10.8
- net at UF14.3: now also UF14.12, UF14.13
- net K12.8: now reaches UK12.8
- net K12.8: now also UK11.2 (A1)
- net at UD14.7 (A7): now also UD10.1
- net at UB5.2 (CP), UC5.2 (CP): now also UB2.2 (CP), UC2.2 (CP)
- net H12.6: now reaches UE11.2
- net H12.6: now also UE10.2
- net at UE12.1: now also R13.2
- net A8.9: now reaches UE12.2
- net at UA15.10: now also UB12.9
- net at UE12.3: now also R12.2
- net at UK13.5 (I1a): now also UJ10.4 (I0), UK10.10, UK10.9
- net at UE7.6 (E3): now also UD4.14 (D5), UD4.4 (D1)
- net at UA1.3 (C): now also UA3.1
- net D7.9: now reaches UA1.4 (~{S})
- net at UA1.5 (Q): now also UA2.1, UA2.2
- net E10.6: now reaches UF13.11 (D3)
- net at UF13.13 (D4): now also UF14.11
- net B12.8: now reaches UF13.3 (D0)
- net at J?.a13 (Pin_a13): no longer UA6.1 (BUS0)
- net at J?.a14 (Pin_a14): no longer UA6.4 (BUS1)
- net at J?.a15 (Pin_a15): no longer UA6.15 (BUS3)
- net at J?.b13 (Pin_b13): now also UA6.1 (BUS0)
- net at J?.b14 (Pin_b14): now also UA6.4 (BUS1)
- net at J?.b15 (Pin_b15): now also UA6.15 (BUS3)
- net DBP: now reaches J?.b29 (Pin_b29)
- net DBP: now also UA13.11
- net at UB7.5: now also UB7.6
- net L11.12: now reaches UK12.5
- net L11.12: now also UK12.6
- net ~{F11.EN}: now reaches UK11.12 (O3)
- net ~{F11.EN}: now also UF11.14 (E)
- net L13.5: now reaches UK11.14 (O1)
- net ~{LOAD.AR.LO}: now reaches UK11.9 (O6)
- net at UE10.3: now also UD12.11
- net at UE10.4: now also UD12.3
- net F13.11: now reaches UE10.6
- net at UC7.2: now also UB8.6
- net at UC7.3: now also UB8.5
- net at UK10.4: now also UK10.5
- net at UE14.4 (~{S}): no longer UE14.10 (~{S})
- net E8.1: now reaches UE14.13 (~{R})
- net H12.14: now reaches UE14.8 (~{Q})
- net at UJ12.11 (I1b): now also UJ13.10 (I0b)
- net K10.11: now reaches UJ12.13 (I3b)
- net R1/R5: now reaches UJ12.4 (I2a)
- net M12.3: now reaches UJ12.9 (Zb)
- net E8.10: now reaches UE11.5
- net E8.10: now also UE14.10 (~{S})
- net ~{LOAD.D9}: now reaches UE6.12 (O3)
- net at UE6.16 (VCC): now also UE6.6 (E3)
- net at UE6.4 (E1): now also UE6.5 (E2), UE6.8 (GND)
- net at UA3.2: now also UA1.11 (C)
- net H12.9: now reaches UE8.5, UE8.6
- net at UJ11.15 (I4): now also UJ11.4 (I0)
- net M12.7: now reaches UJ11.2 (I2)
- net M12.6: now reaches UJ11.5 (Z)
- net ~{A15}: now reaches UC8.4
- net ~{A15}: now also J?.a17 (Pin_a17)
- net at UA15.9: now also UC10.2
- net at UL10.12 (D): now also UM10.11
- net at UM9.3 (C): now also U?.9 (Zc), UL13.4 (C)
- net at UH12.11 (2C): now also UH12.5 (1C)
- net E14.8: now reaches UH12.14 (2~{S2})
- net at UC15.9 (~{PE}): now also UC10.3
- net M8.11: now reaches UF11.9 (Q4)
- net at UA15.12: now also UB11.1
- net T28: now reaches UA15.13
- net B12.1: now reaches UJ13.12 (I2b)
- net at UK12.11: now also UK12.12
- net ~{READ.SWAPPED}: now reaches UD4.12 (Q4)
- net B11.4: now reaches UA1.8 (~{Q})
- net at UA1.9 (Q): now also UA2.4, UA2.5
- net D6.13: now reaches UE14.1 (~{R})
- net at UM8.15 (I2b): now also U?.15 (I2b)
- net at UE10.10: now also UD10.13
- net at UE10.11: now also UD10.10
- net B15.12: now reaches UB11.12
- net P3.13: no longer names the net of UM9.11 (C)
- net P3.13: now also P3.13 (Pin_13)
- net PLCP: no longer names the net of UE5.9 (Cp), UF5.11 (CP), UH5.11 (CP), UJ6.2, UK5.11 (CP), UL5.11 (CP), UM5.11 (CP)
- removed net ~{INT}: UK6.1, UK6.5, UK6.9, UL6.13, UL6.2, UL6.5
- net ~{SWAP.ADR} renamed ~{LOAD.MAR}
- new net: UA2.10, UA2.9
- new net: U?.11 (I0c), UL14.6
- new net: R14.2, UD7.1 (1M), UD7.15 (2M)
- new net: UD12.8, UL13.3 (~{K})
- new net: UA13.1, UA13.8
- new net: UD7.2 (1~{S1}), UD8.8
- new net: R?.2, UM10.2
- new net: UC10.8, UD12.5
- new net: UD12.6, UD7.3 (1~{S2})
- new net: U?.8 (I3a), UM13.11 (Q6), UM14.8 (I3a)
- new net: UM12.7 (Q2), UM13.9 (Q4), UM14.15 (I2b), UM14.6 (I2a)
- new net: UD12.13, UD8.1
- new net: UM10.3, UM10.4
- new net: UB12.13, UB12.2, UC10.10
- new net: UD7.11 (2C), UD7.5 (1C)
- new net: UD7.13 (2~{S1}), UD8.6
- new net: UB8.3, UC7.8
- new net: U?.4 (I1a), UM12.5 (Q1), UM14.4 (I1a)
- new net: P3.7 (Pin_7), U?.12 (O3a)
- new net: P3.6 (Pin_6), U?.14 (O2a)
- new net: P3.5 (Pin_5), U?.16 (O1a)
- new net: P3.3 (Pin_3), U?.18 (O0a)
- new net: U?.2 (I0a), UM14.2 (I0a)
- new net: P3.10 (Pin_10), U?.3 (O3b)
- new net: P3.11 (Pin_11), U?.5 (O2b)
- new net: UC10.6, UD10.8
- new net: P3.1 (Pin_1), UM14.3 (O3b)
- new net: P3.12 (Pin_12), UM14.14 (O2a)
- new net: P3.2 (Pin_2), UM14.17 (I3b), UM14.5 (O2b)
- new net: UA13.6, UA13.9
- new net: UA2.12, UA2.13
- new net A1.10: UD7.7 (1~{Y})
- new net A1.4: UD7.9 (2~{Y})
- new net B15.3: UB12.6
- new net B31: UA13.3
- new net B32: UA14.8
- new net D6.3: UC10.4
- new net F12.5: UM10.10
- new net F13.3: UB12.8
- new net H12.1: UM10.9
- new net IPA12: UB8.4, UC8.11
- new net J13.12: UB12.1
- new net K11.3: UL13.5 (~{S})
- new net M13.12: UA14.12
- new net M8.10: UD8.10, UD8.5
- new net M8.4: UL13.7 (~{Q})
- new net PA?? (21): J?.a21 (Pin_a21), UA8.1 (BUS0)
- new net T11: UA2.11
- new net T30: UA14.11
- new net T6: UA2.3
- new net T7: UA2.6
- new net T8: UA2.8
- new net ~{A??}?: J?.a22 (Pin_a22)
- no-connect marks 1 -> 6
Other:
- moved on the sheet: E15C, UA15A, UA15B, UA15C, UA15F, UA15G, UA1C, UA3A, UA3B, UA3C, UA3D, UA3E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

Commit message: Add more traces, relabeled microcode pipeline register
Parts:
- E15, UA1, UB15, UE14, UE15, UF12, UL10, UM9: value (none) -> 74LS74
- J?: value (none) -> Edge Connector
- P2: value (none) -> Connector
- R13, R14, R9: value (none) -> 1k0
- R? (x2): value (none) -> R
- RN?: value (none) -> 4k7; footprint (none) -> Resistor_THT:R_Array_SIP10
- RN?: value (none) -> 220/330; footprint (none) -> Resistor_THT:R_Array_SIP10
- SW?: value (none) -> SW_DIP_x08
- UA10, UA4, UA5, UA6, UA8, UA9: value (none) -> DS8835
- UA11, UA12: value (none) -> AM2907
- UA13, UM10: value (none) -> 7437
- UA14, UA2: value (none) -> 7438
- UA15, UA3, UC10, UC8, UE12, UJ6: value (none) -> 74LS04
- UA7, UM14, UM6, UM7, UM8: value (none) -> 74LS240
- UB1, UB2, UB5, UB6, UC1, UC15, UC2, UC5, UC6: value (none) -> 74LS669
- UB10, UB9, UD14, UD15: value (none) -> 93L422
- UB11, UE10, UE11: value (none) -> 74LS10
- UB12, UD12, UF14, UK10, UK6, UL14, UL6: value (none) -> 74LS00
- UB13: value (none) -> 6309
- UB4, UC14, UC4, UD6: value (none) -> 74LS157
- UB7, UB8: value (none) -> 74LS30
- UC11, UC12: value (none) -> 74LS173
- UC13, UC9, UM5: value (none) -> 74LS377
- UC7, UD10, UE8, UK12: value (none) -> 74LS02
- UD11, UD9, UJ9, UM12: value (none) -> 74LS378
- UD13: value (none) -> 74LS374
- UD2: value (none) -> 74S139
- UD3: value (none) -> 74S138
- UD4, UE5, UF13: value (none) -> 74LS174
- UD7, UH12: value (none) -> 74120
- UD8, UH13: value (none) -> 74LS20
- UE6, UE7, UH11, UK11: value (none) -> 74LS138
- UF11, UM13: value (none) -> 74LS259
- UF12: renamed from Uf12; value (none) -> 74LS74
- UF6, UJ12, UK13: value (none) -> 74LS153
- UF9: renamed from UF10; value (none) -> AM2901 (0-3)
- UF9: renamed from UF11; value (none) -> AM2901 (4-7)
- UH14: value (none) -> 74LS368
- UH6: value (none) -> 74LS253
- UJ10: value (none) -> 74LS151
- UJ7: renamed from U?; value (none) -> AM2909 (4-7)
- UK7: renamed from U?; value (none) -> AM2909 (0-3)
- UK9: value (none) -> 74S151
- UL11: renamed from U?; value (none) -> 74LS157
- UL13: value (none) -> 74LS109
- UL9: value (none) -> AM2911 (8-10)
- UM15: renamed from U?; value (none) -> 74LS240
- UM3: value (none) -> 76161
- YM11: value (none) -> Crystal
Connections:
- net B15.12 is gone; now on an unnamed net: UB11.12
- net B32 is gone; now on net ~{RESET}: UA14.8
- net M12.10 is gone; now on net CC.L: UK13.6 (I0a)
- net MC16 is gone; now on net PL16: UK5.19 (Q7)
- net MC17 is gone; now on net PL17: UF9.2 (A2), UK5.16 (Q6)
- net MC2 is gone; now on net PL18: UJ11.7 (~{E}), UK9.9 (S2), UM5.6 (Q2), UM6.13 (I1b)
- net MC21 is gone; now on net PL21: UK5.15 (Q5)
- net MC3 is gone; now on net PL19: UJ11.11 (S0), UM5.9 (Q3)
- net MC4 is gone; now on net PL20: UJ11.10 (S1), UJ13.14 (S0), UM5.12 (Q4), UM6.2 (I0a)
- net MC5 is gone; now on net PL21: UJ10.7 (~{E}), UJ13.2 (S1), UM5.15 (Q5)
- net PA?? (23) is gone; now on net PA15: J?.a23 (Pin_a23), UA10.1 (BUS0)
- net T11 is gone; now on net ~{APRE}: UA2.11
- net T6 is gone; now on net ~{RDIN}: UA2.3
- net T7 is gone; now on net ~{WTIN}: UA2.6
- net T8 is gone; now on net ~{DRDY}: UA2.8
- net D6.3: now also UD6.3 (I1a), UF12.12 (D)
- net DP4: now also UA7.12 (O3a), UA7.3 (O3b), UA8.13 (OUT3), UM14.12 (O3a)
- net DP5: now also UA7.14 (O2a), UA7.5 (O2b), UA8.10 (OUT2), UM14.14 (O2a)
- net DP6: now also UA7.16 (O1a), UM14.16 (O1a)
- net DP7: now also UA7.18 (O0a), UA7.9 (O0b), UA8.3 (OUT0), UM14.18 (O0a)
- net GND: now also UD6.15 (E), UD6.8 (GND), UE6.4 (E1), UE6.5 (E2), UE6.8 (GND), UH11.4 (E1), UH11.5 (E2), UH11.8 (GND), UL11.15 (E), UL11.8 (GND)
- net H12.9: now also UD6.11 (I0c), UD6.2 (I0a)
- net K13.11: now also UH13.5
- net K13.4: now also UH13.2
- net K13.5: now also UH13.4
- net M12.7: now also UJ11.13 (I6)
- net PA15: no longer J?.b20 (Pin_b20), UA10.12 (BUS2)
- net S: now also UJ9.14 (D5), UJ9.2 (Q0), UK10.2
- net VCC: now also UD6.16 (VCC), UE6.16 (VCC), UE6.6 (E3), UH11.16 (VCC), UH11.6 (E3)
- net ~{2901.OE}: no longer UL6.8
- net ~{BUSRESET}: now also UF11.15 (Clr), UJ7.15 (~{ZERO})
- net ~{LOAD.DB}: no longer UE6.7 (O7)
- net ~{READ.ILR}: no longer UD5.12 (Q4)
- net ~{READ.SW1}: no longer UA7.1 (OEa), UD5.5 (Q1)
- net at UK12.1: now also UK12.11, UK12.12
- net A15.6: now reaches UA2.10, UA2.9
- net A15.6: now also UA15.6, UC15.7 (~{CEP})
- net E14.1: now reaches UD6.13 (I1d), UD6.6 (I1b)
- net at UD6.14 (I0d): now also UH11.11 (O4)
- net at UD6.5 (I0b): now also UH11.10 (O5)
- net at UE8.13: now also UB12.4
- net ~{LOAD.NSWP}: now reaches UC11.10 (E2), UC11.9 (E1), UC12.10 (E2), UC12.9 (E1)
- net ~{LOAD.NSWP}: now also UH11.7 (O7)
- net K9.7: now reaches UH13.6
- net at UL14.4: now also UL14.5
- net K9.4: now reaches UF12.9 (Q)
- net at UE11.10, UE11.9, UE14.11 (C): now also UE11.12
- net at R?.1, R?.1, UM10.5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: now also UL11.6 (I1b), UM10.13
- net at UB15.2 (D): now also UB15.12 (D)
- net ~{RLE}: now reaches UB15.3 (C)
- net K9.13: now reaches UB15.6 (~{Q})
- net U/~{D}: now reaches UB1.1 (U/~{D}), UB5.1 (U/~{D}), UB6.1 (U/~{D}), UC1.1 (U/~{D}), UC5.1 (U/~{D}), UC6.1 (U/~{D})
- net U/~{D}: now also UF11.7 (Q3)
- net at UM9.10 (~{S}): no longer RN?.7 (R6)
- net at P3.13 (Pin_13), UM9.11 (C): now also RN?.7 (R6)
- net at R?.2, UM10.2: now also UM10.1
- net at UH13.13: now also UK12.13
- net CC.L: now reaches UM14.8 (I3a), UM15.8 (I3a)
- net CC.L: now also UJ10.4 (I0), UK10.10, UK10.9, UM12.10 (Q3); no longer UM13.11 (Q6)
- net CC.F: now reaches UM12.7 (Q2), UM14.6 (I2a)
- net CC.F: now also UM15.6 (I2a); no longer UM13.9 (Q4), UM14.15 (I2b)
- net at UA14.10, UA15.2: now also UA14.9
- net C10.1: now reaches UL11.7 (Zb)
- net ~{PFW}: now reaches UB10.20 (~{WE})
- net ~{PFW}: now also UB9.20 (~{WE})
- net PL21: now reaches UJ9.12 (Q4)
- net PL21: now also UJ13.5 (I1a)
- net K9.14: now reaches UF14.6
- net F11.12: now reaches UE11.13
- net F11.12: now also UM8.17 (I3b)
- net at UD7.14 (2~{S2}): now also UH11.14 (O1)
- net at UA15.10: now also UB12.10; no longer UB12.9
- net ~{LOAD.CC}: now reaches UM12.1 (~{E})
- net ~{LOAD.CC}: now also UE6.7 (O7)
- net CC.V: now reaches UM12.2 (Q0)
- net CC.V: now also UM14.2 (I0a), UM15.2 (I0a)
- net CC.M: now reaches UM12.5 (Q1), UM14.4 (I1a), UM15.4 (I1a)
- net OR3: now reaches UK13.7 (Za)
- net OR2: now reaches UK13.9 (Zb)
- net FP.L: now reaches P3.7 (Pin_7), UM15.12 (O3a)
- net FP.F: now reaches P3.6 (Pin_6), UM15.14 (O2a)
- net at UM15.15 (I2b): no longer UM8.15 (I2b)
- net FP.M: now reaches P3.5 (Pin_5), UM15.16 (O1a)
- net FP.V: now reaches P3.3 (Pin_3), UM15.18 (O0a)
- net at UM15.7 (O1b): now also P3.12 (Pin_12)
- net B11.3: now reaches UA1.6 (~{Q})
- net at UM14.17 (I3b), UM14.5 (O2b): no longer P3.2 (Pin_2)
- net at UH11.13 (O2): now also UC10.9
- net ~{APRE}: now reaches J?.a11 (Pin_a11)
- net INR1: now reaches J?.a13 (Pin_a13)
- net INR1: now also UA7.6 (I2a)
- net INR2: now reaches J?.a14 (Pin_a14)
- net INR2: now also UA7.4 (I1a)
- net INR3: now reaches J?.a15 (Pin_a15)
- net INR3: now also UA7.2 (I0a)
- net INR0: now reaches J?.a16 (Pin_a16)
- net INR0: now also UA7.8 (I3a)
- net ~{RDIN}: now reaches J?.a6 (Pin_a6)
- net ~{WTIN}: now reaches J?.a7 (Pin_a7)
- net ~{DRDY}: now reaches J?.a8 (Pin_a8)
- net ~{DRDY}: now also UA3.3
- net ~{RESET}: now reaches J?.b32 (Pin_b32)
- net K9.1: now reaches UB12.3
- net ~{M13.EN}: now reaches UK11.13 (O2)
- net at UA3.12: now also UH12.13 (2~{S1}), UH12.2 (1~{S1}), UH12.3 (1~{S2})
- net at UA3.13: now also UA3.4
- net K9.3: now reaches UD10.4
- net K9.15: now reaches UD12.1
- net F11.10: now reaches UA13.12
- net L13.4: now reaches UH12.11 (2C), UH12.5 (1C)
- net A13.12: now reaches UF11.10 (Q5)
- net B11.2: now reaches UF11.11 (Q6)
- net M8.17: now reaches UF11.12 (Q7)
- net B12.9: now reaches UF11.4 (Q0)
- net D6.6: now reaches UF11.6 (Q2)
- net B12.3: now reaches UK9.1 (I3)
- net H13.6: now reaches UK9.12 (I7)
- net B15.6: now reaches UK9.13 (I6)
- net F14.6: now reaches UK9.14 (I5)
- net D12.1: now reaches UK9.15 (I4)
- net C13.2: now reaches UK9.2 (I2)
- net D10.4: now reaches UK9.3 (I1)
- net F12.9: now reaches UK9.4 (I0)
- net at UM14.11 (I0b): now also UM13.11 (Q6)
- net F11.11: now reaches UB11.13, UB11.2
- net B11.4: no longer names the net of UA1.8 (~{Q})
- net B15.9 renamed B15.10
- net C15.9: no longer names the net of UB11.6
- net DB3/DB7 renamed R3/7
- net K10.11: no longer names the net of UJ12.13 (I3b)
- net K10.11: now also UK10.11
- net M8.10 renamed M8.12
- net MC0 renamed PL16
- net MC1 renamed PL17
- net MC10 renamed PL26
- net MC11 renamed PL27
- net MC12 renamed PL28
- net MC13 renamed PL29
- net MC14 renamed PL30
- net MC15 renamed PL31
- net MC18 renamed PL18
- net MC19 renamed PL19
- net MC20 renamed PL20
- net MC22 renamed PL22
- net PL22: now also UJ10.11 (S0), UK13.14 (S0), UM5.5 (Q1), UM6.4 (I1a)
- net MC23 renamed PL23
- net PL23: now also UJ10.10 (S1), UK13.2 (S1), UM5.2 (Q0), UM6.8 (I3a)
- net MC26 renamed PL10
- net MC27 renamed PL11
- net MC29 renamed PL13
- net MC31 renamed PL15
- net MC32 renamed PL32
- net MC33 renamed PL33
- net MC37 renamed PL37
- net MC38 renamed PL38
- net MC43 renamed PL43
- net MC44 renamed PL44
- net MC45 renamed PL45
- net MC46 renamed PL46
- net MC47 renamed PL47
- removed net MC6: UJ10.11 (S0), UK13.2 (S1), UM5.5 (Q1), UM6.4 (I1a)
- removed net MC7: UJ10.10 (S1), UK10.11, UK13.14 (S0), UM5.2 (Q0), UM6.8 (I3a)
- net MC8 renamed PL24
- net MC9 renamed PL25
- net PA?? (18) renamed CL0
- net PA?? (19) renamed CL1
- net PA?? (20) renamed CL2
- net PA?? (21) renamed CL3
- net PA?? (24) renamed PA16
- net PA?? (25) renamed PA17
- net T30 renamed T29
- net ~{2909.OE}: no longer names the net of UJ7.22 (~{OE}), UK7.22 (~{OE}), UL9.16 (~{OE})
- net ~{2909.OE}: now also UL6.8
- net ~{READ.SW2} renamed A7.1 (high)
- net A7.1 (high): now also UA7.1 (OEa)
- new net A8.7 (high): UD5.12 (Q4)
- new net F11.4: UB12.9
- new net M14.2 (high): UD5.5 (Q1)
- new net MMIO15: J?.b20 (Pin_b20), UA10.12 (BUS2)
- now unconnected: UK13.5 (I1a)
- no-connect marks 6 -> 7
Other:
- moved on the sheet: R?, UA15E, UA15F, UA2C, UA3B, UA3F, UB11A, UB11B, UB12B, UB15A, UB15B, UC10D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

Commit message: Schematic corrections
Connections:
- net PL16: no longer UK5.19 (Q7)
- net PL17: no longer UF9.2 (A2), UK5.16 (Q6)
- net PL18: no longer UK5.6 (Q2)
- net PL19: no longer UF6.14 (S0), UH6.14 (A0), UK5.9 (Q3)
- net PL20: no longer UK5.12 (Q4)
- net PL21: no longer UK5.15 (Q5)
- net PL22: no longer UK5.5 (Q1), UK6.12
- net PL23: no longer UK5.2 (Q0)
- net ~{PFW}: now also UK11.10 (O5)
- net at UD8.12, UD8.2, UE8.11: no longer UD10.5
- net LSH: now reaches UH6.15 (OEb), UJ6.12
- net (J9.10): now reaches UH6.11 (I1b), UH6.5 (I1a)
- net D10.1: now reaches UD14.7 (A7)
- net D10.1: no longer UD10.1
- net PL53: now reaches UD10.2
- net PL53: now also UK5.15 (Q5)
- net at UD10.3: now also UD10.5
- net D12.10: now reaches UH12.1 (1M)
- net K9.7 renamed K9.12
- net RAM7: no longer names the net of UH6.10 (I0b)
- net ~{LD.SR} renamed ~{LD.FLR}
- new net D14.7: UD10.1
- new net PL48: UK5.19 (Q7)
- new net PL49: UF9.2 (A2), UK5.16 (Q6)
- new net PL50: UK5.6 (Q2)
- new net PL51: UF6.14 (S0), UH6.14 (A0), UK5.9 (Q3)
- new net PL52: UK5.12 (Q4)
- new net PL54: UK5.5 (Q1), UK6.12
- new net PL55: UK5.2 (Q0)
- no-connect marks 7 -> 8
Other:
- moved on the sheet: UD10A, UD10B

Commit message: Pins from today's beeping
Parts:
- added JP1: (no value), symbol oldchips:Jumper_3_Bridged23
- added R18: (no value), symbol Device:R
- added R19: 4k7, symbol Device:R
- added RN?: 220/330, Resistor_THT:R_Array_SIP10, symbol Device:R_Network_Dividers_x08_SIP
- UC8: value 74LS04 -> (none)
- gave numbers to parts that had none: 1
- renumbered UF9 to UF7
Connections:
- net CLK is gone; now on net B31: UF7.15 (CP)
- net (F7): no longer UC9.18 (D7)
- net A10: now also UC7.6
- net A11: now also UC8.1
- net A12: now also UA3.9, UB10.21 (A4); no longer UC7.6
- net A13: now also UA3.5
- net A14: now also UA3.11, UB10.6 (A6)
- net A15: now also UB10.7 (A7)
- net A9: now also UC7.5
- net B31: now also P1.b31 (Pin_b31)
- net DP0: now also UA9.3 (OUT0)
- net DP1: now also UA9.6 (OUT1); no longer UC12.4 (Q1)
- net DP2: now also UC12.3 (Q0)
- net DP3: now also UA9.10 (OUT2)
- net DP4: now also UA10.3 (OUT0)
- net DP5: now also UA10.6 (OUT1)
- net DP6: now also UC11.3 (Q0), UC12.14 (D0), UD13.5 (O1)
- net DP7: now also UA10.10 (OUT2)
- net DP?: no longer UC12.3 (Q0)
- net F0: now also UC9.3 (D0)
- net F1: now also UC9.4 (D1)
- net F11.10: now also UA13.13
- net F4: now also UC9.13 (D4)
- net F6: now also UC9.17 (D6)
- net F7: now also UC9.18 (D7)
- net GND: now also UB10.19 (~{CS1}), UB10.8 (GND), UC11.15 (Mr), UC11.8 (GND), UC12.15 (Mr), UC15.10 (~{CET}), UC15.3 (P0), UC15.4 (P1), UC15.5 (P2), UC15.6 (P3), UC15.8 (GND), UF12.7 (GND), RN?.1 (COM1)
- net INR0: now also RN?.5 (R4)
- net INR1: now also RN?.2 (R1)
- net INR2: now also RN?.3 (R2)
- net INR3: now also RN?.4 (R3)
- net IPA12: no longer UB8.4
- net IPA14: now also UB8.11
- net J13.12: now also UB8.8
- net M13.12: now also UA14.13
- net PL28: now also UL9.20 (PUP)
- net PL55: now also UC14.1 (S)
- net VCC: now also UB10.17 (CS2), UB10.22 (VCC), UB15.1 (~{R}), UB15.13 (~{R}), UB15.4 (~{S}), UC15.1 (U/~{D}), UC15.16 (VCC), UF12.14 (VCC), RN?.10 (COM2); no longer R12.1, R13.1, R14.1
- net ~{2901.OE}: now also UL6.8
- net ~{A13}: now also UA3.6
- net ~{A??}: no longer P1.a10 (Pin_a10)
- net ~{RE}: no longer UL9.3 (~{RE})
- net at UE8.13: now also UB12.5; no longer UB12.4
- net ~{A12}: now reaches UA3.8
- net ~{A12}: now also P1.a10 (Pin_a10)
- net READ.SWP: now reaches UC11.1 (Oe1), UC12.1 (Oe1)
- net READ.SWP: now also UC11.2 (Oe2), UC12.2 (Oe2)
- net at UJ6.8, UJ7.25 (~{FE}): now also UL9.19 (~{FE})
- net E15.5: now reaches UA14.1
- net E15.5: now also UA14.2
- net at UA13.1, UA13.8: now also UA13.2
- net ~{WAR.OVR}: now reaches UC10.13
- net at UB11.6: now also UC10.3, UC15.9 (~{PE})
- net at UJ7.22 (~{OE}), UK7.22 (~{OE}), UL9.16 (~{OE}): now also UJ6.10; no longer UL6.8
- net at UA14.4: now also UA14.5, UB10.10 (Q0)
- net at UA14.6: now also P1.a26 (Pin_a26)
- net IPA13: now reaches UC7.12
- net IPA13: now also UB8.12
- net at UB12.13, UB12.2: now also UC10.11, JP1.3 (B), R19.2; no longer UC10.10
- net IPA18: now reaches UC8.5
- net IPA18: now also UB8.1
- net at UC8.6: now also JP1.2 (C)
- net at UB10.11 (D1): now also UC9.16 (Q6)
- net at UB10.13 (D2): now also UC9.15 (Q5)
- net at UB10.15 (D3): now also UC9.12 (Q4)
- net E12.4: now reaches UB10.18 (~{OE})
- net at UB10.9 (D0): now also UC9.19 (Q7)
- net at UC9.6 (Q2): now also UB9.11 (D1)
- net T27: now reaches UA15.11
- net T27: now also P1.a27 (Pin_a27), RN?.9 (R8)
- net IPA11: now reaches UB8.3, UC7.8
- net IPA11: now also UB8.2
- net at UC7.4: now also UB7.2
- net at UA13.10: now also UA13.6, UA13.9
- net at UB7.4: now also JP1.1 (A), R18.2
- net C10.11: now reaches UB7.8
- net IPA15: now reaches UB8.6, UC7.2
- net IPA16: now reaches UB8.5, UC7.3
- net ~{A14}: now reaches UA3.10
- net at UC14.11 (I0c): now also UC13.15 (Q5)
- net at UC14.15 (E): now also UC14.8 (GND)
- net WAR.OVR: now reaches UC5.15 (~{TC})
- net at UC13.4 (D1): now also UB13.9 (D3)
- net A15.4: now reaches UC15.2 (CP)
- net L10.7: now reaches UC10.1
- net at UA2.12, UA2.13: now also UC10.10
- net F14.10 renamed F14.9
- net ~{A??}? renamed ~{A11}
- new net A1.5: UB12.4
- new net IPA17: UB8.4
- no-connect marks 8 -> 12
Other:
- moved on the sheet: UA14B, UA15F, UA2D, UA3C, UA3D, UA3E, UB11A, UB12B, UB15A, UB15B, UC10E, UC7B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

Commit message: Errors corrected
Parts:
- removed UE14: 74LS74, symbol 74xx:74LS74
- added R?: (no value), symbol Device:R
- added UE14: (no value), symbol 74xx:74LS04
Connections:
- net T22 is gone; now on net ~{A11}: UC8.2
- net ~{A??} is gone; now on net ~{A14}: P1.a9 (Pin_a9)
- net D6.3: no longer UD6.3 (I1a), UF12.12 (D)
- net E8.10: now also UE14.10
- net F4: now also UD9.3 (D0)
- net GND: now also UC14.15 (E), UC14.8 (GND), UE14.7 (GND)
- net H12.6: now also UE14.2; no longer UE10.2
- net IPA11: now also UA9.2 (IN0), UB9.16 (Q3)
- net IPA12: now also UA9.5 (IN1), UB9.14 (Q2)
- net IPA13: now also UA9.14 (IN3), UB9.12 (Q1)
- net IPA14: now also UA9.11 (IN2), UB9.10 (Q0)
- net IPA17: now also UA10.14 (IN3), UB10.12 (Q1), UB11.9
- net IPA18: now also UA14.4, UA14.5, UB10.10 (Q0)
- net VCC: now also UE14.14 (VCC)
- net at UE15.3 (C): now also UE14.3
- net at UE15.4 (~{S}): now also UE14.12
- net A14.1: now reaches UE15.5 (Q)
- net ~{A4}: now reaches P1.b9 (Pin_b9), UA5.1 (BUS0)
- net ~{A7}: now reaches P1.b12 (Pin_b12), UA5.12 (BUS2)
- net ~{A6}: now reaches P1.b11 (Pin_b11), UA5.15 (BUS3)
- net ~{A5}: now reaches P1.b10 (Pin_b10), UA5.4 (BUS1)
- net at UE11.10, UE11.12, UE11.9: now also UE14.11
- net E14.9: now reaches UE11.11
- net E14.9: now also UE14.9
- net at UK6.9: now also UK6.1, UK6.5, UL6.13, UL6.2, UL6.5, R?.2
- net at UE8.1: now also UE14.13; no longer UE11.1
- net D6.1: now reaches UB15.10 (~{S})
- net E11.6: now reaches UB15.11 (C)
- net ~{A0}: now reaches P1.b5 (Pin_b5), UA4.1 (BUS0)
- net ~{A3}: now reaches P1.b8 (Pin_b8), UA4.12 (BUS2)
- net ~{A2}: now reaches P1.b7 (Pin_b7), UA4.15 (BUS3)
- net ~{A1}: now reaches P1.b6 (Pin_b6), UA4.4 (BUS1)
- net at UB12.12: now also JP1.3 (B), R19.2
- net B7.8: now reaches UB12.13, UB12.2, UC10.11
- net B7.8: no longer JP1.3 (B), R19.2
- net at UB10.14 (Q2), UB11.10: now also UA10.5 (IN1)
- net at UE15.11 (C): now also UE14.6
- net B10.19: now reaches UE12.4
- net ~{A8}: now reaches P1.b13 (Pin_b13), UA6.1 (BUS0)
- net ~{A9}: now reaches P1.b14 (Pin_b14), UA6.4 (BUS1)
- net ~{A10}: now reaches P1.b15 (Pin_b15), UA6.15 (BUS3)
- net at UE11.3: now also UE10.2
- net B15.11: now reaches UE11.6
- net D9.5: now reaches UC14.10 (I1c)
- net D9.2: now reaches UC14.13 (I1d)
- net D9.12: now reaches UC14.3 (I1a)
- net D9.15: now reaches UC14.6 (I1b)
- net JSR?: now reaches UK9.6 (~{Z})
- net JSR?: now also R?.1
- net A15.6: no longer names the net of UA15.6, UA2.10, UA2.9, UC15.7 (~{CEP})
- net E14.1 renamed F11.6
- net F11.6: now also UE14.1
- net E14.8: no longer names the net of UH12.14 (2~{S2})
- net E14.8: now also UE14.8
- net L10.7 renamed L11.7
- new net C10.4: UD6.3 (I1a), UF12.12 (D)
Other:
- moved on the sheet: UE8C, UH14, UL6C
