File: kicad/CPU6.kicad_sch (KiCad schematic)
At the start: 140 parts, among them P1 Edge Connector, P2 Connector, P3 Connector

Commit message: Redo schematic
Parts:
- removed R?: (no value), symbol Device:R
- removed R? (x2): R, symbol Device:R
- removed RN?: 4k7, Resistor_THT:R_Array_SIP10, symbol Device:R_Network09
- removed RN? (x2): 220/330, Resistor_THT:R_Array_SIP10, symbol Device:R_Network_Dividers_x08_SIP
- removed SW?: SW_DIP_x08, symbol Switch:SW_DIP_x08
- removed YM11: Crystal, symbol Device:Crystal
- added C1, C10, C11, C12, C13, C14, C15, C16, C17, C18, C19, C2, C20, C21, C22, C23, C24, C25, C26, C27, C28, C29, C3, C30, C31, C32, C33, C34, C35, C36, C37, C38, C4, C40, C41, C42, C43, C44, C45, C46, C47, C48, C49, C5, C50, C51, C54, C6, C7, C8, C9: 0.1uF, symbol Device:C
- added C39: C_Polarized_US, symbol Device:C_Polarized_US
- added C52, C53: 150uF, symbol Device:C_Polarized_US
- added CR1: D_Filled, symbol Device:D_Filled
- added DSWI556: SW_DIP_x08, symbol Switch:SW_DIP_x08
- added P10, P4, P8: Conn_02x08_Counter_Clockwise, symbol Connector_Generic:Conn_02x08_Counter_Clockwise
- added P5, P6: Conn_02x25_Odd_Even, symbol Connector_Generic:Conn_02x25_Odd_Even
- added P7: Conn_02x07_Counter_Clockwise, symbol Connector_Generic:Conn_02x07_Counter_Clockwise
- added R1, R2, R3, R5, R8: R, symbol Device:R
- added R10, R11, R17, R6: 1k0, symbol Device:R
- added R15: 10k, symbol Device:R
- added R16, R4: 220/330, Resistor_THT:R_Array_SIP10, symbol Device:R_Network_Dividers_x08_SIP
- added R7: 4k7, Resistor_THT:R_Array_SIP10, symbol Device:R_Network09
- added XTAL556: Crystal, symbol Device:Crystal
- JP1: value (none) -> Jumper_3_Bridged23
- R12, R13: value 1k0 -> 4k7
- R18: value (none) -> 4k7
- UC8, UE14: value (none) -> 74LS04
- UF9: value AM2901 (0-3) -> AM2901
- UJ7: value AM2909 (4-7) -> AM2909
- UK7: value AM2909 (0-3) -> AM2909
Connections:
- net (F1) is gone; now on net F1: UB13.7 (D1), UC13.8 (D3), UD11.4 (D1)
- net (F7) is gone; now on net F7: UB13.14 (D7), UC13.18 (D7)
- net (J9.10) is gone; now on net FLR.C: UH6.11 (I1b), UH6.5 (I1a)
- net A1.5 is gone; now on net RDIN: UB12.4
- net A8.9 is gone; now on an unnamed net: UE12.2
- net ADR.CLK is gone; now on an unnamed net: UC6.2 (CP), UD6.4 (Za)
- net B10.19 is gone; now on an unnamed net: UE12.4
- net B11.3 is gone; now on net ~{RDIN1}: UA1.6 (~{Q})
- net B11.5 is gone; now on net ~{WTIN1}: UF12.3 (C)
- net B12.3 is gone; now on net NOT.MEM: UK9.1 (I3)
- net B12.9 is gone; now on net INT.EN: UF11.4 (Q0)
- net B15.10 is gone; now on net DMA.EN: UD6.1 (S)
- net B15.11 is gone; now on net E11.6: UE11.6
- net B15.3 is gone; now on net ~{RLE}: UB12.6
- net C is gone; now on net ALU.C: UH6.3 (I3a)
- net C10.11 is gone; now on net ~{REG}: UB7.8
- net C13.2 is gone; now on net RIR.0: UK9.2 (I2)
- net C15.2 is gone; now on net ~{PHI1}': UA15.4
- net D10.1 is gone; now on an unnamed net: UD14.7 (A7)
- net D12.10 is gone; now on net E14.10: UH12.1 (1M)
- net D14.7 is gone; now on an unnamed net: UD10.1
- net D6.1 is gone; now on net DMA.EN: UB15.10 (~{S})
- net D6.3 is gone; now on net ~{BUSY}: UC10.4
- net D7.7 is gone; now on net ~{WT}: UA1.10 (~{S}), UF12.4 (~{S})
- net D7.9 is gone; now on net ~{RD}: UA1.4 (~{S})
- net D9.12 is gone; now on net CL3: UC14.3 (I1a)
- net D9.15 is gone; now on net CL2: UC14.6 (I1b)
- net D9.2 is gone; now on net CL0: UC14.13 (I1d)
- net D9.5 is gone; now on net CL1: UC14.10 (I1c)
- net E12.4 is gone; now on an unnamed net: UB10.18 (~{OE})
- net E14.9 is gone; now on net E8.13: UE11.11, UE14.9
- net E8.10 is gone; now on net E14.10: UE11.5, UE14.10
- net F11.10 is gone; now on net PARO: UA13.12, UA13.13
- net F11.11 is gone; now on net PE.EN: UB11.13, UB11.2
- net F11.4 is gone; now on net INT.EN: UB12.9
- net F11.6 is gone; now on net INC.DMA: UD6.13 (I1d), UD6.6 (I1b), UE14.1
- net F12.3 is gone; now on net ~{WTIN1}: UB11.4, UB11.5
- net F13.11 is gone; now on net E10.6: UE10.6
- net F13.3 is gone; now on an unnamed net: UB12.8
- net H12.1 is gone; now on net E14.10: UM10.9
- net H12.6 is gone; now on an unnamed net: UE11.2, UE14.2
- net H14.2 is gone; now on net ~{LVL15}: UE10.8, UF14.2
- net IPA11 is gone; now on net PA11: UA9.2 (IN0), UB8.2, UB8.3, UB9.16 (Q3), UC7.8
- net IPA12 is gone; now on net PA12: UA9.5 (IN1), UB9.14 (Q2), UC8.11
- net IPA13 is gone; now on net PA13: UA9.14 (IN3), UB8.12, UB9.12 (Q1), UC7.12
- net IPA14 is gone; now on net PA14: UA9.11 (IN2), UB8.11, UB9.10 (Q0), UC7.11
- net IPA15 is gone; now on net PA15: UB8.6, UC7.2
- net IPA16 is gone; now on net PA16: UB8.5, UC7.3
- net IPA17 is gone; now on net PA17: UA10.14 (IN3), UB10.12 (Q1), UB11.9, UB8.4
- net IPA18 is gone; now on net PA18: UA14.4, UA14.5, UB10.10 (Q0), UB8.1, UC8.5
- net J13.12 is gone; now on net ~{BAD.PG}: UB12.1, UB8.8
- net K13.11 is gone; now on net LVL15.Q: UF13.12 (Q4), UH13.5
- net K13.12 is gone; now on net E10.6.Q: UF13.10 (Q3)
- net K13.4 is gone; now on net DMA13.Q: UF13.5 (Q1), UH13.2
- net K13.5 is gone; now on net INTR.Q: UF13.2 (Q0), UH13.4
- net K9.1 is gone; now on net NOT.MEM: UB12.3
- net K9.12 is gone; now on net INT: UH13.6
- net K9.13 is gone; now on net PE: UB15.6 (~{Q})
- net K9.14 is gone; now on an unnamed net: UF14.6
- net K9.15 is gone; now on net B12.11: UD12.1
- net K9.3 is gone; now on an unnamed net: UD10.4
- net K9.4 is gone; now on an unnamed net: UF12.9 (Q)
- net L11.12 is gone; now on net PHI2: UK12.5, UK12.6
- net L11.7 is gone; now on net PHI1: UC10.1
- net L13.4 is gone; now on net ~{PHI1}: UH12.11 (2C), UH12.5 (1C)
- net L13.5 is gone; now on net ~{K11.O1}: UK11.14 (O1)
- net L15.11 is gone; now on an unnamed net: UM7.17 (I3b)
- net LB0 is gone; now on net ALU.B0: UF11.13 (D), UF9.17 (B0)
- net LB1 is gone; now on net ALU.B1: UF11.1 (A0), UF9.18 (B1)
- net LB2 is gone; now on net ALU.B2: UF11.2 (A1), UF9.19 (B2)
- net LB3 is gone; now on net ALU.B3: UF11.3 (A2), UF9.20 (B3)
- net M10.10 is gone; now on an unnamed net: UF12.5 (Q)
- net M12.3 is gone; now on net CC.V: UJ12.9 (Zb)
- net M12.6 is gone; now on net CC.F: UJ11.5 (Z)
- net M13.12 is gone; now on net IACK: UA14.12, UA14.13
- net M13.6 is gone; now on net TIMER.EN: UF14.10
- net M14.2 (high) is gone; now on net ~{READ.CCR}: UD5.5 (Q1)
- net M7.4 is gone; now on net DIP.H: UF14.1
- net M8.11 is gone; now on net DMA.EN: UF11.9 (Q4)
- net M8.17 is gone; now on net DMA.RD: UF11.12 (Q7)
- net M8.4 is gone; now on net L13.7: UL13.7 (~{Q})
- net M9.9 is gone; now on net TIMER: UF14.9
- net PL37 is gone; now on net ALU.I3: UH5.15 (Q5)
- net PL38 is gone; now on net ALU.I4: UH5.5 (Q1)
- net PL43 is gone; now on net ALU.B0: UF5.9 (Q3)
- net PL44 is gone; now on net ALU.B1: UF5.12 (Q4)
- net PL45 is gone; now on net ALU.B2: UF5.15 (Q5)
- net PL46 is gone; now on net ALU.B3: UF5.5 (Q1)
- net PL47 is gone; now on net ALU.A0: UF5.2 (Q0), UF7.4 (A0)
- net PL48 is gone; now on net ALU.A1: UK5.19 (Q7)
- net PL49 is gone; now on net ALU.A2: UF9.2 (A2), UK5.16 (Q6)
- net PL50 is gone; now on net ALU.A3: UK5.6 (Q2)
- net Q0 is gone; now on net ALU.Q0: UH6.4 (I2a)
- net R1/R5 is gone; now on net R6: UJ12.4 (I2a)
- net R3/7 is gone; now on net R4: UJ10.15 (I4)
- net T28 is gone; now on net ~{PE}: UA15.13
- net T29 is gone; now on net ~{IACK}: UA14.11
- net Z is gone; now on net ALU.Z: UF9.11 (F=0), UJ9.3 (D0)
- net ~{LOAD.AR.LO} is gone; now on net ~{LOAD.ALO}: UK11.9 (O6)
- net ~{LOAD.D9} is gone; now on net ~{LOAD.CL}: UE6.12 (O3)
- net ~{LOAD.DB} is gone; now on net ~{RLE}: UA11.1 (~{RLE}), UA12.1 (~{RLE})
- net ~{LOAD.PTBR} is gone; now on net ~{LOAD.MAP}: UE6.11 (O4)
- net ~{M13.EN} is gone; now on net ~{STATE2.EN}: UK11.13 (O2)
- net ~{READ.ILR} is gone; now on net ~{READ.MSR}: UA8.7 (~{R}), UH14.1 (OEa)
- net ~{READ.SW1} is gone; now on net ~{READ.INR}: UM7.1 (OEa)
- net ~{READ.SWAPPED} is gone; now on net ~{READ.SWP}: UD4.12 (Q4)
- net ~{REG.READ} is gone; now on net ~{READ.RF}: UD13.1 (OE)
- net ~{RESET} is gone; now on net ~{MRST}: P1.b32 (Pin_b32), UA14.8
- net A11: now also UB9.1 (A3)
- net A12: now also UB9.21 (A4)
- net A13: now also UA7.15 (I2b), UB9.5 (A5)
- net A14: now also UA7.13 (I1b), UB9.6 (A6)
- net A15: now also UB9.7 (A7)
- net A5: no longer UA5.5 (IN1)
- net CC.F: now also UM12.6 (D2); no longer UM12.7 (Q2), UM14.6 (I2a), UM15.6 (I2a)
- net CC.L: now also UJ10.5 (Z), UM12.11 (D3); no longer UJ10.4 (I0), UK10.10, UK10.9, UK13.6 (I0a), UM12.10 (Q3), UM14.8 (I3a), UM15.8 (I3a)
- net CC.M: now also UJ12.7 (Za), UM12.4 (D1); no longer UM12.5 (Q1), UM14.4 (I1a), UM15.4 (I1a)
- net CC.V: now also UM12.3 (D0); no longer UM12.2 (Q0), UM14.2 (I0a), UM15.2 (I0a)
- net CL0: now also UA8.14 (IN3), UD9.2 (Q0); no longer P1.a18 (Pin_a18), UA8.15 (BUS3)
- net CL1: now also UA8.11 (IN2), UD10.9, UD9.5 (Q1); no longer P1.a19 (Pin_a19), UA8.12 (BUS2)
- net CL2: now also UA8.5 (IN1), UD10.12, UD9.15 (Q5); no longer P1.a20 (Pin_a20), UA8.4 (BUS1)
- net CL3: now also UA8.2 (IN0), UD10.11, UD9.12 (Q4); no longer P1.a21 (Pin_a21), UA8.1 (BUS0)
- net D12.1: now also P10.8 (Pin_8); no longer UK9.15 (I4)
- net DBP: no longer P1.b29 (Pin_b29)
- net DP0: now also UK7.5 (R0), UM6.3 (O3b), UM7.12 (O3a), UM7.9 (O0b); no longer UA4.3 (OUT0)
- net DP1: now also UC12.5 (Q2), UH14.7 (O3a), UK7.4 (R1); no longer UA4.6 (OUT1)
- net DP2: now also UK7.3 (R2); no longer UA4.13 (OUT3)
- net DP3: now also UK7.2 (R3), UM6.9 (O0b), UM7.18 (O0a), UM7.3 (O3b); no longer UA4.10 (OUT2)
- net DP4: now also UJ7.5 (R0), UM6.12 (O3a)
- net DP5: now also UC12.12 (D2), UJ7.4 (R1), UM6.14 (O2a)
- net DP6: now also UA10.13 (OUT3), UA7.7 (O1b), UA8.6 (OUT1), UJ7.3 (R2), UM6.16 (O1a); no longer UD13.5 (O1)
- net DP7: now also UJ7.2 (R3), UM6.18 (O0a)
- net F0: now also UB13.6 (D0), UC13.3 (D0), UD11.6 (D2), P4.3 (Pin_3)
- net F2: now also UB13.8 (D2), UC13.7 (D2), UD11.3 (D0), P4.5 (Pin_5)
- net F3: now also UB13.9 (D3), UC13.4 (D1), P4.6 (Pin_6)
- net F4: now also UA12.17 (IN3), UB13.11 (D4), UC13.13 (D4), P4.10 (Pin_10)
- net F5: now also UB13.12 (D5), UC13.14 (D5), P4.11 (Pin_11)
- net F6: now also UB13.13 (D6), UC13.17 (D6), UD13.5 (O1), UD9.14 (D5), P4.12 (Pin_12)
- net F7: now also UD9.13 (D4), P4.13 (Pin_13)
- net GND: now also P1.a1 (Pin_a1), P1.a36 (Pin_a36), P1.b1 (Pin_b1), P1.b36 (Pin_b36), P2.14 (Pin_14), P2.15 (Pin_15), P2.16 (Pin_16), P2.17 (Pin_17), P2.18 (Pin_18), P2.19 (Pin_19), P2.20 (Pin_20), P2.21 (Pin_21)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
- net JSR?: now also UK6.1, UK6.5, UK6.9, UL6.13, UL6.2, UL6.5, R8.2; no longer UK9.6 (~{Z})
- net M8.12: now also UD8.4, UM8.12 (O3a)
- net MMIO15: now also UA10.11 (IN2), UC8.12; no longer P1.b20 (Pin_b20), UA10.12 (BUS2)
- net OR2: now also UK7.8 (OR2)
- net OR3: now also UK7.6 (OR3)
- net PA11: no longer P1.b16 (Pin_b16), UA9.1 (BUS0)
- net PA12: now also UC7.9, P10.2 (Pin_2); no longer P1.b17 (Pin_b17), UA9.4 (BUS1)
- net PA13: no longer P1.b18 (Pin_b18), UA9.15 (BUS3)
- net PA14: now also P10.4 (Pin_4); no longer P1.b19 (Pin_b19), UA9.12 (BUS2)
- net PA15: now also UA10.2 (IN0), UB10.16 (Q3), UB11.11, P10.5 (Pin_5); no longer P1.a23 (Pin_a23), UA10.1 (BUS0)
- net PA16: now also UA10.5 (IN1), UB10.14 (Q2), UB11.10, P10.6 (Pin_6); no longer P1.a24 (Pin_a24), UA10.4 (BUS1)
- net PA17: now also P10.7 (Pin_7); no longer P1.a25 (Pin_a25), UA10.15 (BUS3)
- net PL16: now also UK7.13 (D0)
- net PL17: now also UK7.11 (D1)
- net PL18: now also UK7.9 (D2)
- net PL19: now also UK7.7 (D3), UM6.11 (I0b)
- net PL20: now also UJ7.13 (D0)
- net PL21: now also UJ7.11 (D1), UM6.4 (I1a); no longer UJ13.5 (I1a), UJ9.12 (Q4)
- net PL22: now also UJ7.9 (D2), UM6.6 (I2a); no longer UM6.4 (I1a)
- net PL23: now also UJ7.7 (D3)
- net PL24: now also UJ10.9 (S2), UL9.7 (D0)
- net PL25: now also UL9.6 (D1)
- net PL26: now also UL9.5 (D2)
- net PL28: now also UK7.26 (PUP)
- net PL32: now also UJ6.5, UK6.4
- net PL52: now also UF6.2 (S1), UH6.2 (A1)
- net U/~{D}: now also UB2.1 (U/~{D}), UC2.1 (U/~{D})
- net VCC: now also P1.a2 (Pin_a2), P1.a35 (Pin_a35), P1.b2 (Pin_b2), P1.b35 (Pin_b35), P3.22 (Pin_22), P3.23 (Pin_23), P3.24 (Pin_24), P3.25 (Pin_25), P3.26 (Pin_26), R12.1, R13.1, R14.1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
- net WAR.OVR: now also UC10.12, UD12.9; no longer UC5.15 (~{TC})
- net ~{A12}: now also P1.a9 (Pin_a9); no longer P1.a10 (Pin_a10)
- net ~{A14}: now also P1.a10 (Pin_a10); no longer P1.a9 (Pin_a9)
- net ~{DRDY}: now also UA14.3, R16.9 (R8)
- net BUSY: now reaches UD6.10 (I1c)
- net BUSY: now also UB11.6, UC10.3, UC15.9 (~{PE})
- net ~{INC.MAR}: now reaches UD6.14 (I0d)
- net ~{INC.MAR}: now also UH11.10 (O5); no longer UH11.11 (O4)
- net ~{INC.WAR}: now reaches UD6.5 (I0b)
- net ~{INC.WAR}: now also UH11.11 (O4); no longer UH11.10 (O5)
- net at UD6.9 (Zc): now also UB2.2 (CP), UB5.2 (CP), UC2.2 (CP), UC5.2 (CP)
- net MC17: now reaches UM3.10 (D1), UM5.17 (D6)
- net MC17: now also P6.33 (Pin_33)
- net MC18: now reaches UM3.11 (D2), UM5.7 (D2)
- net MC18: now also P6.35 (Pin_35)
- net MC19: now reaches UM3.13 (D3), UM5.8 (D3)
- net MC19: now also P6.37 (Pin_37)
- net MC20: now reaches UM3.14 (D4), UM5.13 (D4)
- net MC20: now also P6.39 (Pin_39)
- net MC21: now reaches UM3.15 (D5), UM5.14 (D5)
- net MC21: now also P6.41 (Pin_41)
- net MC22: now reaches UM3.16 (D6), UM5.4 (D1)
- net MC22: now also P6.43 (Pin_43)
- net MC23: now reaches UM3.17 (D7), UM5.3 (D0)
- net MC23: now also P6.45 (Pin_45)
- net at UM3.18 (CE3): now also UE3.18 (CE3), UF3.18 (CE3), UH3.18 (CE3), UJ3.18 (CE3), UK3.18 (CE3), UL3.18 (CE3), R11.2
- net at UM3.19 (CE2): now also UE3.19 (CE2), UF3.19 (CE2), UH3.19 (CE2), UJ3.19 (CE2), UK3.19 (CE2), UL3.19 (CE2), R10.2
- net MC16: now reaches UM3.9 (D0), UM5.18 (D7)
- net MC16: now also P6.31 (Pin_31)
- net E14.10: now reaches UD8.12, UD8.2, UE8.11
- net E14.10: now also UD12.10
- net ~{BUS.WAIT}: now reaches UE7.12 (O3), UE8.12
- net E8.13: now reaches UB12.5, UE8.13
- net DIP.1: now reaches UM7.11 (I0b)
- net DIP.1: now also DSWI556.4, R7.7 (R6)
- net DIP.2: now reaches UM7.13 (I1b)
- net DIP.2: now also P3.8 (Pin_8), DSWI556.3, R4.3 (R2); no longer UM7.6 (I2a)
- net DIP.3: now reaches UM7.15 (I2b)
- net DIP.3: now also DSWI556.2, R7.6 (R5)
- net ~{READ.CCR}: now reaches UM14.1 (OEa), UM7.19 (OEb)
- net DIP.R: now reaches UM7.2 (I0a)
- net DIP.R: now also UL10.2 (D), UL10.9 (Q), UL11.13 (I1d), UM10.12, DSWI556.5, P7.13 (Pin_13), R7.3 (R2)
- net at R9.2, UL10.1 (~{R}), UL10.13 (~{R}): no longer UL11.1 (S)
- net at UC11.11 (D3): now also UC12.6 (Q3)
- net at UC11.13 (D1): now also UC12.4 (Q1)
- net ~{XX.CLK}': now reaches UC11.7 (Cp)
- net ~{XX.CLK}': now also UC12.7 (Cp), UC13.11 (CP), UC9.11 (CP), UD11.9 (C), UD13.11 (Cp), UD4.9 (Cp), UD5.9 (Cp), UD9.9 (C), UE5.9 (Cp), UE8.2, UE8.4
- net P7.2: now reaches UL14.4, UL14.5
- net P7.2: now also UL11.5 (I0b), P7.2 (Pin_2)
- net at UJ6.8, UJ7.25 (~{FE}), UL9.19 (~{FE}): now also UK7.25 (~{FE})
- net E10.12: now reaches UE14.3, UE15.3 (C)
- net E10.12: now also UA1.3 (C), UA3.1, UE10.12
- net P7.12: now reaches UJ6.11
- net P7.12: now also P7.12 (Pin_12), R7.2 (R1)
- net DMA7: now reaches P2.7 (Pin_7)
- net DMA7: now also R7.8 (R7)
- net ~{XX.CLK}: now reaches UF12.11 (C), UF13.9 (Cp)
- net ~{XX.CLK}: now also UF7.15 (CP), UF9.15 (CP), UJ9.9 (C), UK10.6, UK11.4 (E1), UK11.5 (E2)
- net XX.CLK: now reaches UJ6.1
- net XX.CLK: now also UE10.13, UE8.5, UE8.6, UH12.10 (2Y), UK10.4, UK10.5
- net ~{XX.CLK}'': now reaches UF5.11 (CP), UH5.11 (CP), UJ6.2, UK5.11 (CP), UL5.11 (CP), UM5.11 (CP)
- net ~{XX.CLK}'': now also UJ5.11 (CP), UJ7.27 (CP), UK7.27 (CP), UL9.1 (CP); no longer UE5.9 (Cp)
- net at UL11.6 (I1b), UM10.13: now also UL10.5 (Q); no longer UM10.5
- net 15MHz: now reaches UL11.3 (I1a), UM10.6
- net 15MHz: now also R3.2, XTAL556.2
- net at UE14.5: now also UE14.4
- net ALU.A3: now reaches UF9.1 (A3)
- net ALU.A3: now also UF7.1 (A3)
- net at UF9.16 (Q3_RO/LI): now also UF7.21 (Q0_LO/RI)
- net ALU.Q0: now reaches UF9.21 (Q0_LO/RI), UH6.9 (Zb), UJ10.12 (I7)
- net ALU.A1: now reaches UF9.3 (A1)
- net ALU.A1: now also UF7.3 (A1)
- net ALU.A0: now reaches UF9.4 (A0)
- net ALU.RAM0: now reaches UF7.16 (Q3_RO/LI), UF9.9 (RAM0_LO/RI), UJ10.13 (I6)
- net MC52: now reaches UK3.14 (D4), UK5.13 (D4)
- net MC52: now also P5.47 (Pin_47)
- net MC53: now reaches UK3.15 (D5), UK5.14 (D5)
- net MC53: now also P5.49 (Pin_49)
- net MC49: now reaches UK3.10 (D1), UK5.17 (D6)
- net MC49: now also P5.41 (Pin_41)
- net MC48: now reaches UK3.9 (D0), UK5.18 (D7)
- net MC48: now also P5.39 (Pin_39)
- net MC55: now reaches UK3.17 (D7), UK5.3 (D0)
- net MC55: now also P5.48 (Pin_48)
- net MC54: now reaches UK3.16 (D6), UK5.4 (D1)
- net MC54: now also P5.50 (Pin_50)
- net MC50: now reaches UK3.11 (D2), UK5.7 (D2)
- net MC50: now also P5.43 (Pin_43)
- net MC51: now reaches UK3.13 (D3), UK5.8 (D3)
- net MC51: now also P5.45 (Pin_45)
- net ~{PA18}': now reaches UD8.13
- net ~{PA18}': now also JP1.2 (C), UC8.6, UD12.4, UJ13.4 (I2a)
- net DMA11: now reaches UD8.9
- net DMA11: now also P2.11 (Pin_11), UD12.2, UM8.6 (I2a), R4.9 (R8)
- net R1: now reaches UB3.10 (I1c), UB4.10 (I1c)
- net R1: now also UB9.13 (D2), UC9.5 (Q1), UD15.13 (D2)
- net R0: now reaches UB4.13 (I1d)
- net R0: now also UB3.13 (I1d), UB9.15 (D3), UC9.2 (Q0), UD15.15 (D3)
- net R3: now reaches UB3.3 (I1a), UB4.3 (I1a)
- net R3: now also UB9.9 (D0), UC9.9 (Q3), UD15.9 (D0)
- net R2: now reaches UB3.6 (I1b), UB4.6 (I1b)
- net R2: now also UB9.11 (D1), UC9.6 (Q2), UD15.11 (D1)
- net ~{LOAD.SAR}: now reaches UK7.1 (~{RE})
- net ~{LOAD.SAR}: now also UE6.9 (O6)
- net ~{RESET1}: now reaches UK7.15 (~{ZERO})
- net ~{RESET1}: now also UA1.1 (~{R}), UA1.13 (~{R}), UD4.5 (Q1), UF11.15 (Clr), UJ7.15 (~{ZERO}), UL9.9 (~{ZERO}), UM13.15 (Clr)
- net ~{PA18}: now reaches P1.a26 (Pin_a26), UA14.6
- net ~{PA18}: now also R16.7 (R6)
- net 60Hz: now reaches P3.13 (Pin_13), UM9.11 (C)
- net 60Hz: now also R4.7 (R6)
- net ~{TIMER.RESET}: now reaches UM13.10 (Q5), UM9.13 (~{R})
- net at UM10.1, UM10.2: now also R2.1, XTAL556.1
- net DMA9: now reaches P2.9 (Pin_9), UM10.8
- net P7.5: now reaches UL10.10 (~{S}), UL10.4 (~{S})
- net P7.5: now also P7.5 (Pin_5), R17.2
- net DMA10: now reaches P2.10 (Pin_10), UM8.8 (I3a)
- net DMA10: now also R4.8 (R7)
- net DMA6: now reaches UM8.3 (O3b)
- net DMA6: now also P2.6 (Pin_6); no longer P2.11 (Pin_11)
- net DMA12: now reaches P2.12 (Pin_12)
- net DMA12: now also R4.6 (R5)
- net DMA13: now reaches P2.13 (Pin_13)
- net DMA13: now also UF13.4 (D1), R4.5 (R4)
- net DMA2: now reaches P2.2 (Pin_2), UM8.9 (O0b)
- net DMA3: now reaches P2.3 (Pin_3), UM8.7 (O1b)
- net DMA4: now reaches P2.4 (Pin_4), UM8.5 (O2b)
- net DMA5: now reaches P2.5 (Pin_5), UM8.16 (O1a)
- net DMA8: now reaches P2.8 (Pin_8), UM8.18 (O0a)
- net E8.1: now reaches UE14.13, UE8.1
- net ~{E7.O1}: now reaches UE7.14 (O1), UE8.3
- net B15.9: now reaches UB15.9 (Q)
- net B15.9: now also UE10.5
- net ALU.B1: now reaches UM13.1 (A0)
- net ALU.B1: now also UF7.18 (B1)
- net at UM14.11 (I0b): no longer UM13.11 (Q6)
- net IACK: now reaches UM13.12 (Q7)
- net ALU.B0: now reaches UM13.13 (D)
- net ALU.B0: now also UF7.17 (B0)
- net ~{STATE2.EN}: now reaches UM13.14 (E)
- net ALU.B2: now reaches UM13.2 (A1)
- net ALU.B2: now also UF7.19 (B2)
- net ALU.B3: now reaches UM13.3 (A2)
- net ALU.B3: now also UF7.20 (B3)
- net M13.O0: now reaches UM13.4 (Q0)
- net M13.O0: now also UM8.13 (I1b)
- net M13.O1: now reaches UM13.5 (Q1)
- net M13.O1: now also UM8.15 (I2b)
- net TIMER.EN: now reaches UM13.6 (Q2)
- net RUN: now reaches UM13.9 (Q4)
- net RUN: now also UM14.15 (I2b)
- net at UD13.13 (D4): now also UD15.16 (Q3)
- net at UA15.1: now also C39.1, CR1.2 (A), R15.2
- net R5: now reaches UC3.10 (I1c), UC4.10 (I1c)
- net R5: now also UB10.13 (D2), UC9.15 (Q5), UD14.13 (D2), UJ11.15 (I4), UJ11.4 (I0)
- net R4: now reaches UC3.13 (I1d)
- net R4: now also UB10.15 (D3), UC4.13 (I1d), UC9.12 (Q4), UD14.15 (D3)
- net R7: now reaches UC3.3 (I1a), UC4.3 (I1a)
- net R7: now also UB10.9 (D0), UC9.19 (Q7), UD14.9 (D0), UJ12.12 (I2b)
- net R6: now reaches UC3.6 (I1b), UC4.6 (I1b)
- net R6: now also UB10.11 (D1), UC9.16 (Q6), UD14.11 (D1)
- net NOT.MEM: now reaches UD12.12
- net M8.14: now reaches UD12.13, UD8.1
- net M8.14: now also UE11.4, UM8.14 (O2a)
- net at UJ7.16 (S0), UL9.10 (S0): now also UK6.3
- net at UM10.3, UM10.4: now also UM10.5, R2.2, R3.1
- net PL4: now reaches UE5.10 (Q3), UE6.1 (A0)
- net MC4: now reaches UE3.14 (D4), UE5.11 (D3)
- net MC4: now also P6.7 (Pin_7)
- net PL6: now reaches UE5.12 (Q4), UE6.3 (A2)
- net MC6: now reaches UE3.16 (D6), UE5.13 (D4)
- net MC6: now also P6.11 (Pin_11)
- net MC7: now reaches UE3.17 (D7), UE5.14 (D5)
- net MC7: now also P6.13 (Pin_13)
- net PL5: now reaches UE5.2 (Q0), UE6.2 (A1)
- net MC5: now reaches UE3.15 (D5), UE5.3 (D0)
- net MC5: now also P6.9 (Pin_9)
- net at UC5.4 (P1): now also UC4.9 (Zc); no longer UC4.7 (Zb)
- net at UC5.5 (P2): now also UC4.7 (Zb); no longer UC4.9 (Zc)
- net PHI2: now reaches UL11.12 (Zd)
- net P7.8: now reaches UL11.14 (I0d)
- net P7.8: now also P7.8 (Pin_8)
- net P7.3: now reaches UL11.2 (I0a)
- net P7.3: now also P7.3 (Pin_3)
- net ~{PHI1}: now reaches UL11.9 (Zc), UL13.4 (C), UM9.3 (C)
- net ~{PHI1}: now also UD7.11 (2C), UD7.5 (1C)
- net P7.4: now reaches UL10.12 (D), UM10.11
- net P7.4: now also P7.4 (Pin_4)
- net B12.11: now reaches UB12.11
- net B12.11: now also UK9.15 (I4)
- net MC41: now reaches UF3.10 (D1), UF5.17 (D6)
- net MC41: now also P5.25 (Pin_25)
- net MC42: now reaches UF3.11 (D2), UF5.7 (D2)
- net MC42: now also P5.27 (Pin_27)
- net MC43: now reaches UF3.13 (D3), UF5.8 (D3)
- net MC43: now also P5.29 (Pin_29)
- net MC44: now reaches UF3.14 (D4), UF5.13 (D4)
- net MC44: now also P5.31 (Pin_31)
- net MC45: now reaches UF3.15 (D5), UF5.14 (D5)
- net MC45: now also P5.33 (Pin_33)
- net MC46: now reaches UF3.16 (D6), UF5.4 (D1)
- net MC46: now also P5.35 (Pin_35)
- net MC47: now reaches UF3.17 (D7), UF5.3 (D0)
- net MC47: now also P5.37 (Pin_37)
- net MC40: now reaches UF3.9 (D0), UF5.18 (D7)
- net MC40: now also P5.23 (Pin_23)
- net FLR.C: now reaches UF6.4 (I2a)
- net FLR.C: now also UJ10.2 (I2), UJ9.10 (Q3)
- net MAP2: now reaches UB10.2 (A2), UD11.2 (Q0)
- net MAP2: now also UB9.2 (A2), UM15.17 (I3b)
- net MAP1: now reaches UB10.3 (A1), UD11.5 (Q1)
- net MAP1: now also UB9.3 (A1), UM15.15 (I2b)
- net MAP0: now reaches UB10.4 (A0), UD11.7 (Q2)
- net MAP0: now also UB9.4 (A0), UM15.13 (I1b)
- net MC28: now reaches UL3.14 (D4), UL5.13 (D4)
- net MC28: now also P5.2 (Pin_2)
- net MC29: now reaches UL3.15 (D5), UL5.14 (D5)
- net MC29: now also P5.1 (Pin_1)
- net MC25: now reaches UL3.10 (D1), UL5.17 (D6)
- net MC25: now also P6.49 (Pin_49)
- net MC24: now reaches UL3.9 (D0), UL5.18 (D7)
- net MC24: now also P6.47 (Pin_47)
- net MC31: now reaches UL3.17 (D7), UL5.3 (D0)
- net MC31: now also P5.5 (Pin_5)
- net MC30: now reaches UL3.16 (D6), UL5.4 (D1)
- net MC30: now also P5.3 (Pin_3)
- net MC26: now reaches UL3.11 (D2), UL5.7 (D2)
- net MC26: now also P6.50 (Pin_50)
- net MC27: now reaches UL3.13 (D3), UL5.8 (D3)
- net MC27: now also P6.48 (Pin_48)
- net MC36: now reaches UH3.14 (D4), UH5.13 (D4)
- net MC36: now also P5.15 (Pin_15)
- net MC37: now reaches UH3.15 (D5), UH5.14 (D5)
- net MC37: now also P5.17 (Pin_17)
- net MC33: now reaches UH3.10 (D1), UH5.17 (D6)
- net MC33: now also P5.9 (Pin_9)
- net MC32: now reaches UH3.9 (D0), UH5.18 (D7)
- net MC32: now also P5.7 (Pin_7)
- net MC39: now reaches UH3.17 (D7), UH5.3 (D0)
- net MC39: now also P5.21 (Pin_21)
- net MC38: now reaches UH3.16 (D6), UH5.4 (D1)
- net MC38: now also P5.19 (Pin_19)
- net MC34: now reaches UH3.11 (D2), UH5.7 (D2)
- net MC34: now also P5.11 (Pin_11)
- net MC35: now reaches UH3.13 (D3), UH5.8 (D3)
- net MC35: now also P5.13 (Pin_13)
- net ALU.RAM3: now reaches UF7.8 (RAM3_RO/LI), UH6.7 (Za), UJ10.14 (I5)
- net P7.9: now reaches UL6.9
- net P7.9: now also P7.9 (Pin_9), R7.10 (R9)
- net ALU.C: now reaches UJ9.11 (D3)
- net ALU.C: now also UF7.33 (Cn+4)
- net FLR.S: now reaches UJ12.3 (I3a), UJ9.5 (Q1)
- net FLR.S: now also UJ12.5 (I1a), UJ13.6 (I0a)
- net FLR.V: now reaches UJ11.9 (S2), UJ9.7 (Q2)
- net FLR.V: now also UJ13.11 (I1b)
- net DMA13.Q: now reaches UF14.4
- net DMA13.Q: now also UF14.5, UK13.4 (I2a)
- net at UC14.12 (Zd), UD14.1 (A3): now also UD15.1 (A3)
- net at UC14.9 (Zc), UD14.2 (A2): now also UD15.2 (A2)
- net at UC13.5 (Q1), UD14.21 (A4): now also UD15.21 (A4)
- net at UC14.7 (Zb), UD14.3 (A1): now also UD15.3 (A1)
- net at UC14.4 (Za), UD14.4 (A0): now also UD15.4 (A0)
- net at UC13.6 (Q2), UD14.5 (A5): now also UD15.5 (A5)
- net at UC13.9 (Q3), UD14.6 (A6): now also UD15.6 (A6)
- net ~{LOAD.ALO}: now reaches UB2.9 (~{PE}), UC2.9 (~{PE})
- net P4.14: now reaches R13.2, UE12.1
- net P4.14: now also P4.14 (Pin_14)
- net MC9: now reaches UJ3.10 (D1), UJ5.17 (D6)
- net MC9: now also P6.17 (Pin_17)
- net MC10: now reaches UJ3.11 (D2), UJ5.7 (D2)
- net MC10: now also P6.19 (Pin_19)
- net MC11: now reaches UJ3.13 (D3), UJ5.8 (D3)
- net MC11: now also P6.21 (Pin_21)
- net MC12: now reaches UJ3.14 (D4), UJ5.13 (D4)
- net MC12: now also P6.23 (Pin_23)
- net MC13: now reaches UJ3.15 (D5), UJ5.14 (D5)
- net MC13: now also P6.25 (Pin_25)
- net MC14: now reaches UJ3.16 (D6), UJ5.4 (D1)
- net MC14: now also P6.27 (Pin_27)
- net MC15: now reaches UJ3.17 (D7), UJ5.3 (D0)
- net MC15: now also P6.29 (Pin_29)
- net MC8: now reaches UJ3.9 (D0), UJ5.18 (D7)
- net MC8: now also P6.15 (Pin_15)
- net ~{BUS.RD}: now reaches UD7.14 (2~{S2}), UH11.14 (O1)
- net MC1: now reaches UD2.3 (A1), UD3.2 (A1), UE3.10 (D1)
- net MC1: now also P6.1 (Pin_1)
- net MC2: now reaches UD3.3 (A2), UE3.11 (D2)
- net MC2: now also P6.3 (Pin_3)
- net MC3: now reaches UD2.1 (E), UD3.6 (E3), UE3.13 (D3)
- net MC3: now also P6.5 (Pin_5)
- net MC0: now reaches UD2.2 (A0), UD3.1 (A0), UE3.9 (D0)
- net MC0: now also P6.2 (Pin_2)
- net ~{LOAD.MAP}: now reaches UD11.1 (~{E})
- net P4.7: now reaches R12.2, UE12.3
- net INT.EN: now reaches UK13.10 (I0b)
- net INT.EN: now also UC10.5
- net LVL15.Q: now reaches UK13.11 (I1b)
- net E10.6.Q: now reaches UK13.12 (I2b)
- net INTR.Q: now reaches UK13.5 (I1a)
- net ~{MRST}: now reaches UD4.14 (D5), UD4.4 (D1), UE7.6 (E3)
- net FP.MAP2: now reaches P3.10 (Pin_10), UM15.3 (O3b)
- net FP.MAP1: now reaches P3.11 (Pin_11), UM15.5 (O2b)
- net FP.MAP0: now reaches P3.12 (Pin_12), UM15.7 (O1b)
- net RDIN: now reaches UA1.5 (Q), UA2.1, UA2.2
- net FP.HALT: now reaches P3.1 (Pin_1), UM14.3 (O3b)
- net R/F: now reaches P3.15 (Pin_15)
- net R/F: now also UL14.12, UL14.13, R4.4 (R3)
- net FP.ABT: now reaches P3.16 (Pin_16)
- net FP.ABT: now also R1.2
- net FP.RUN: now reaches P3.2 (Pin_2)
- net FP.RUN: now also UM14.17 (I3b), UM14.5 (O2b)
- net FP.DELAY: now reaches P3.9 (Pin_9)
- net FP.DELAY: now also UH14.6 (I3)
- net ~{BUS.WT}: now reaches UC10.9, UH11.13 (O2)
- net X.CLK: now reaches UE10.2, UE11.3
- net X.CLK: now also UH12.6 (1Y)
- net ~{PE}: now reaches P1.a28 (Pin_a28)
- net ~{PE}: now also R16.8 (R7)
- net ~{IACK}: now reaches P1.a29 (Pin_a29)
- net at P1.a30 (Pin_a30): now also P1.a31 (Pin_a31), P1.a32 (Pin_a32), P1.a33 (Pin_a33)
- net at UB7.5, UB7.6: now also UC8.8
- net FLR.16Z: now reaches UJ12.13 (I3b), UK10.11
- net FLR.Z: now reaches UJ12.11 (I1b), UJ13.10 (I0b)
- net FLR.Z: now also UJ9.14 (D5), UJ9.2 (Q0), UK10.2
- net CC.M.Q: now reaches UJ12.6 (I0a)
- net CC.M.Q: now also UM12.5 (Q1), UM14.4 (I1a), UM15.4 (I1a)
- net at UB1.2 (CP), UC1.2 (CP): now also UB6.2 (CP)
- net RIR.0: now reaches UD10.3, UD10.5
- net RIR.0: now also UC13.2 (Q0)
- net RIR.4: now reaches UC13.12 (Q4), UC14.14 (I0d)
- net RIR.4: now also UD10.6
- net M9.5: now reaches UM8.2 (I0a), UM9.5 (Q)
- net ~{XX.CLK}''': now reaches UH12.9 (2~{Y})
- net ~{XX.CLK}''': now also UD6.11 (I0c), UD6.2 (I0a)
- net PA18: now reaches UH14.10 (I4)
- net ~{LVL15}: now reaches UH14.2 (I1)
- net ALU.Z: now reaches UF7.11 (F=0)
- net ALU.Z: now also R5.2
- net ALU.A2: now reaches UF7.2 (A2)
- net ~{WTIN1}: now reaches UA1.8 (~{Q})
- net ABT: now reaches UM14.13 (I1b)
- net ABT: now also UM13.11 (Q6)
- net at UM14.7 (O1b): now also R1.1
- net DMA.EN: now reaches UM8.11 (I0b)
- net L13.7: now reaches UM8.4 (I1a)
- net M14.9: now reaches UE10.9
- net A1.10 renamed ~{WT}
- net A1.4 renamed ~{RD}
- net A1.6 renamed ~{RDIN1}
- net A13.12 renamed PARO
- net A15.4 renamed ~{PHI1}'
- net A7.1 (high) renamed ~{READ.INR}
- net A8.7 (high) renamed ~{READ.MSR}
- net B11.2 renamed PE.EN
- net B12.1 renamed ~{BAD.PG}
- net B12.8: no longer names the net of UF13.3 (D0)
- net B15.6 renamed PE
- net B31 renamed ~{BUSCLK}
- net ~{BUSCLK}: no longer UF7.15 (CP)
- net B7.8 renamed ~{REG}
- net C10.1 renamed PHI1
- net C10.4 renamed ~{BUSY}
- net D10.4: no longer names the net of UK9.3 (I1)
- net D6.6 renamed INC.DMA
- net DP?: no longer names the net of UC11.6 (Q3)
- net DP?: no longer UC12.5 (Q2)
- net E6.12 renamed ~{LOAD.CL}
- net E7.2 renamed PL14
- net F11.12 renamed DMA.RD
- net F12.5: no longer names the net of UM10.10
- net F12.9: no longer names the net of UK9.4 (I0)
- net F14.1 renamed DIP.H
- net DIP.H: now also DSWI556.6, R7.4 (R3)
- net F14.6: no longer names the net of UK9.14 (I5)
- net F14.9 renamed TIMER
- net H11.3 renamed PL12
- removed net H12.9: UD6.11 (I0c), UD6.2 (I0a), UE8.5, UE8.6
- net H13.12 renamed PL9
- net H13.6 renamed INT
- net HALFCARRY renamed ALU.HC
- net INR0 renamed ~{INR0}
- net ~{INR0}: now also R16.5 (R4)
- net INR1 renamed ~{INR1}
- net ~{INR1}: now also R16.4 (R3)
- net INR2 renamed ~{INR2}
- net ~{INR2}: now also R16.3 (R2)
- net INR3 renamed ~{INR3}
- net ~{INR3}: now also R16.2 (R1)
- net K11.3 renamed ~{K11.O1}
- net K12.8 renamed PL8
- net K12.9 renamed PL7
- net LI0 renamed ALU.I0
- net LI1 renamed ALU.I1
- net LI2 renamed ALU.I2
- net LI3 renamed ALU.I3
- net LI4 renamed ALU.I4
- net LI5 renamed ALU.I5
- net LI6 renamed ALU.I6
- net LI7 renamed ALU.I7
- net LI8 renamed ALU.I8
- net LSH: no longer names the net of UH6.15 (OEb), UJ6.12
- net M12.7 renamed CC.F.Q
- net CC.F.Q: now also UM12.7 (Q2), UM14.6 (I2a), UM15.6 (I2a)
- net READ.SWP renamed ~{READ.SWP}
- net S renamed ALU.S
- net ALU.S: no longer UJ9.14 (D5), UJ9.2 (Q0), UK10.2
- net T27 renamed ~{INTR}
- net UA0 renamed MCA0
- net MCA0: now also P8.4 (Pin_4)
- net UA1 renamed MCA1
- net MCA1: now also P8.3 (Pin_3)
- net UA10 renamed MCA10
- net MCA10: now also P8.6 (Pin_6)
- net UA2 renamed MCA2
- net MCA2: now also P8.12 (Pin_12)
- net UA3 renamed MCA3
- net MCA3: now also P8.8 (Pin_8)
- net UA4 renamed MCA4
- net MCA4: now also P8.7 (Pin_7)
- net UA5 renamed MCA5
- net MCA5: now also P8.13 (Pin_13)
- net UA6 renamed MCA6
- net UA7 renamed MCA7
- net MCA7: now also P8.10 (Pin_10)
- net UA8 renamed MCA8
- net MCA8: now also P8.9 (Pin_9)
- net UA9 renamed MCA9
- net MCA9: now also P8.5 (Pin_5)
- net V renamed ALU.V
- net ~{2901.OE}: no longer names the net of UF7.40 (~{OE}), UF9.40 (~{OE}), UL6.8
- net ~{A0} renamed AB0
- net ~{A10} renamed AB10
- net ~{A1} renamed AB1
- net ~{A2} renamed AB2
- net ~{A3} renamed AB3
- net ~{A4} renamed AB4
- net ~{A5} renamed AB5
- net ~{A6} renamed AB6
- net ~{A7} renamed AB7
- net ~{A8} renamed AB8
- net ~{A9} renamed AB9
- net ~{ADR.CEP}: no longer names the net of UB1.7 (~{CEP}), UB6.7 (~{CEP}), UC1.7 (~{CEP}), UC6.7 (~{CEP}), UD6.7 (Zb)
- net ~{BUSRESET} renamed ~{RESET2}
- net ~{RESET2}: no longer UA1.1 (~{R}), UA1.13 (~{R}), UF11.15 (Clr), UJ7.15 (~{ZERO})
- net ~{CONST} renamed ~{READ.CONST}
- net ~{F11.EN} renamed ~{STATE1.EN}
- net ~{LD.AR.HI} renamed ~{LOAD.AHI}
- net ~{LD.FLR} renamed ~{LOAD.FLR}
- net ~{LOAD.CC} renamed ~{LOAD.CCR}
- net ~{LOAD.DR} renamed ~{LOAD.DBR}
- net ~{LOAD.MXR} renamed ~{LOAD.RR}
- net ~{LOAD.NSWP} renamed ~{LOAD.SWP}
- net ~{PFW} renamed ~{WRITE.PF}
- net ~{PROME} renamed ALU/~{PROM}
- net ~{READ.ADR.HI} renamed ~{READ.AHI}
- net ~{READ.ADR.LO} renamed ~{READ.ALO}
- net ~{READ.PA} renamed ~{READ.PF}
- net ~{REG.RD} renamed ~{READ.RF}
- net ~{REG.WE} renamed ~{WRITE.RF}
- net ~{RE}: no longer names the net of UJ7.1 (~{RE})
- net ~{RE}: no longer UE6.9 (O6)
- net ~{WAR.OVR}: no longer names the net of UC10.13
- net ~{WAR.OVR}: now also UC5.15 (~{TC})
- net ~{WK.CEP}: no longer names the net of UB2.7 (~{CEP}), UB5.7 (~{CEP}), UC2.7 (~{CEP}), UC5.7 (~{CEP}), UD6.12 (Zd)
- new net: R8.1, UK9.6 (~{Z})
- new net: P10.10 (Pin_10), P10.11 (Pin_11), P10.12 (Pin_12)
- new net CC.L.Q: UJ10.4 (I0), UK10.10, UK10.9, UK13.6 (I0a), UM12.10 (Q3), UM14.8 (I3a), UM15.8 (I3a)
- new net CC.V.Q: UM12.2 (Q0), UM14.2 (I0a), UM15.2 (I0a)
- new net DBP???: P1.b29 (Pin_b29)
- new net DIP.0: DSWI556.8
- new net DIP.I: DSWI556.7, R7.5 (R4), UM7.6 (I2a)
- new net DIP.M: DSWI556.1
- new net FLR.HC: UJ13.5 (I1a), UJ9.12 (Q4)
- new net P7.1: P7.1 (Pin_1), R6.2, UL11.1 (S)
- new net P7.6: P7.6 (Pin_6)
- new net P7.7: P7.7 (Pin_7)
- new net ~{CL0}: P1.a18 (Pin_a18), UA8.15 (BUS3)
- new net ~{CL1}: P1.a19 (Pin_a19), UA8.12 (BUS2)
- new net ~{CL2}: P1.a20 (Pin_a20), UA8.4 (BUS1)
- new net ~{CL3}: P1.a21 (Pin_a21), UA8.1 (BUS0)
- new net ~{MMIO15}: P1.b20 (Pin_b20), UA10.12 (BUS2)
- new net ~{PA11}: P1.b16 (Pin_b16), UA9.1 (BUS0)
- new net ~{PA12}: P1.b17 (Pin_b17), UA9.4 (BUS1)
- new net ~{PA13}: P1.b18 (Pin_b18), UA9.15 (BUS3)
- new net ~{PA14}: P1.b19 (Pin_b19)
- new net ~{PA15}: P1.a23 (Pin_a23), UA10.1 (BUS0)
- new net ~{PA16}: P1.a24 (Pin_a24), UA10.4 (BUS1)
- new net ~{PA17}: P1.a25 (Pin_a25), UA10.15 (BUS3)
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Other:
- note added: "0-3"
- note added: "4-7"
- note added: "47uF?"
- note added: "8-10"
- note added: "Bad Page or Register File access"
- note added: "DMA start?"
- note added: "DMA?"
- note added: "FAULT/OVERFLOW"
- note added: "LINK/CARRY"
- note added: "LSH"
- note added: "MINUS/SIGN and VALUE/ZERO"
- note added: "READ.CCR - CCR High, Sense Switches Low READ.INR - INR High, Other Dip Switches Low READ.MSR - CL High, H14 Low"
- note added: "RSH"
- note added: "read or write"
- title: (none) -> Centurion CPU6

Commit message: 99.9% traces; functional image
Parts:
- C1, C10, C11, C12, C13, C14, C15, C16, C17, C18, C19, C2, C20, C21, C22, C23, C24, C25, C26, C27, C28, C29, C3, C30, C31, C32, C33, C34, C35, C36, C37, C38, C4, C40, C41, C42, C43, C44, C45, C46, C47, C48, C49, C5, C50, C51, C54, C6, C7, C8, C9: footprint (none) -> Capacitor_THT:C_Disc_D3.0mm_W1.6mm_P2.50mm
- C39: footprint (none) -> Capacitor_THT:CP_Axial_L25.0mm_D10.0mm_P30.00mm_Horizontal
- C52, C53: footprint (none) -> Capacitor_THT:CP_Axial_L34.5mm_D20.0mm_P41.00mm_Horizontal
- CR1: footprint (none) -> Diode_THT:D_DO-201AD_P15.24mm_Horizontal
- DSW1: renamed from DSWI556; footprint (none) -> Package_DIP:DIP-16_W7.62mm
- JP1: footprint (none) -> Connector_PinHeader_2.54mm:PinHeader_1x03_P2.54mm_Vertical
- P1: footprint (none) -> Connector_PinHeader_2.54mm:PinHeader_2x36_P2.54mm_Vertical
- P10, P4, P8: footprint (none) -> Connector_PinSocket_2.54mm:PinSocket_2x08_P2.54mm_Horizontal
- P2, P3: footprint (none) -> Connector_IDC:IDC-Header_2x13_P2.54mm_Horizontal
- P5, P6: footprint (none) -> Connector_IDC:IDC-Header_2x25_P2.54mm_Vertical
- P7: footprint (none) -> Connector_PinSocket_2.54mm:PinSocket_2x07_P2.54mm_Horizontal
- R1: value R -> 220R; footprint (none) -> Resistor_THT:R_Axial_DIN0309_L9.0mm_D3.2mm_P12.70mm_Horizontal
- R10, R11, R12, R13, R14, R15, R17, R18, R19, R6, R9: footprint (none) -> Resistor_THT:R_Axial_DIN0309_L9.0mm_D3.2mm_P12.70mm_Horizontal
- R2, R3: value R -> 330R; footprint (none) -> Resistor_THT:R_Axial_DIN0309_L9.0mm_D3.2mm_P12.70mm_Horizontal
- R5: value R -> 470R; footprint (none) -> Resistor_THT:R_Axial_DIN0309_L9.0mm_D3.2mm_P12.70mm_Horizontal
- R8: value R -> 47R; footprint (none) -> Resistor_THT:R_Axial_DIN0309_L9.0mm_D3.2mm_P12.70mm_Horizontal
- UA1, UA13, UA14, UA15, UA2, UA3, UB11, UB12, UB15, UB7, UB8, UC10, UC7, UC8, UD10, UD12, UD8, UE10, UE11, UE12, UE14, UE15, UE8, UF12, UF14, UH13, UJ6, UK10, UK12, UK6, UL10, UL14, UL6, UM10, UM9: footprint (none) -> Package_DIP:DIP-14_W7.62mm
- UA10, UA4, UA5, UA6, UA8, UA9, UB1, UB2, UB3, UB4, UB5, UB6, UC1, UC11, UC12, UC14, UC15, UC2, UC3, UC4, UC5, UC6, UD11, UD2, UD3, UD4, UD5, UD6, UD7, UD9, UE5, UE6, UE7, UF11, UF13, UF6, UH11, UH12, UH14, UH6, UJ10, UJ11, UJ12, UJ13, UJ9, UK11, UK13, UK9, UL11, UL13, UM12, UM13: footprint (none) -> Package_DIP:DIP-16_W7.62mm
- UA11, UA12, UA7, UB13, UC13, UC9, UD13, UF5, UH5, UJ5, UK5, UL5, UM14, UM15, UM5, UM6, UM7, UM8: footprint (none) -> Package_DIP:DIP-20_W7.62mm
- UB10, UB9, UD14, UD15: footprint (none) -> Package_DIP:DIP-22_W7.62mm
- UE15: renamed from E15; footprint (none) -> Package_DIP:DIP-14_W7.62mm
- UE3, UF3, UH3, UJ3, UK3, UL3, UM3: footprint (none) -> Package_DIP:DIP-24_W7.62mm
- UF7: value AM2901 (4-7) -> AM2901; footprint (none) -> Package_DIP:DIP-40_W15.24mm
- UF9: footprint (none) -> Package_DIP:DIP-40_W15.24mm
- UJ7, UK7: footprint (none) -> Package_DIP:DIP-28_W7.62mm
- UL9: value AM2911 (8-10) -> AM2911; footprint (none) -> Package_DIP:DIP-20_W7.62mm
- XTAL1: renamed from XTAL556; footprint (none) -> Crystal:Crystal_DS15_D1.5mm_L5.0mm_Horizontal
Connections:
- net D12.1 is gone; now on net B12.11: P10.8 (Pin_8)
- net DBP??? is gone; now on net DBPO: P1.b29 (Pin_b29)
- net DIP.0 is gone; now on net DIP.O: DSW1.8
- net E15.5 is gone; now on net BUS.READY: UA14.1, UA14.2
- net P7.6 is gone; now on net GND: P7.6 (Pin_6)
- net P7.7 is gone; now on net GND: P7.7 (Pin_7)
- net ~{MRST} is gone; now on net DIP.M: P1.b32 (Pin_b32), UA14.8, UD4.14 (D5), UD4.4 (D1), UE7.6 (E3)
- net ~{XX.CLK} is gone; now on net ~{CPU.CLKC}: UF12.11 (C), UF13.9 (Cp), UF7.15 (CP), UF9.15 (CP), UJ9.9 (C), UK10.6, UK11.4 (E1), UK11.5 (E2)
- net A11: now also P10.16 (Pin_16)
- net A12: now also P10.15 (Pin_15), UA7.17 (I3b)
- net A13: now also P10.14 (Pin_14)
- net A14: now also P10.13 (Pin_13)
- net A15: now also P10.10 (Pin_10), P10.11 (Pin_11), P10.12 (Pin_12), UA7.11 (I0b)
- net A5: now also UA5.5 (IN1)
- net CC.V.Q: now also UJ12.10 (I0b)
- net DIP.R: no longer P7.13 (Pin_13), UL10.2 (D), UL10.9 (Q), UL11.13 (I1d), UM10.12
- net DMA12: now also UM14.11 (I0b)
- net DP0: now also UA4.3 (OUT0), UC11.11 (D3), UC12.6 (Q3)
- net DP1: now also UA4.6 (OUT1), UD13.15 (O5)
- net DP2: now also UA4.13 (OUT3), UD13.16 (O6)
- net DP3: now also UA4.10 (OUT2), UC11.13 (D1), UC12.4 (Q1), UD13.19 (O7)
- net DP4: now also UA9.13 (OUT3), UC11.6 (Q3), UC12.11 (D3)
- net DP5: now also UD13.6 (O2)
- net DP6: now also UD13.5 (O1)
- net DP7: now also UC11.4 (Q1), UC12.13 (D1), UD13.2 (O0)
- net E11.6: now also UM9.4 (~{S})
- net F0: now also UA11.17 (IN3)
- net F1: now also P4.4 (Pin_4), UA11.13 (IN2)
- net F2: now also UA11.7 (IN1)
- net F3: now also UA11.3 (IN0)
- net F5: now also UA12.13 (IN2)
- net F6: now also UA12.7 (IN1); no longer UD13.5 (O1)
- net F7: now also UA12.3 (IN0)
- net FP.DELAY: now also R4.2 (R1)
- net GND: now also P4.1 (Pin_1), P4.15 (Pin_15), P4.16 (Pin_16), P4.2 (Pin_2), P7.10 (Pin_10), P7.11 (Pin_11), P8.1 (Pin_1), P8.2 (Pin_2), UA4.9 (~{W}), UA5.9 (~{W}), UJ7.10 (OR1), UJ7.12 (OR0), UJ7.6 (OR3), UJ7.8 (OR2), UL13.2 (J), UL9.4 (D3), UM14.19 (OEb), UM15.1 (OEa), UM15.19 (OEb), UM8.1 (OEa), UM8.19 (OEb), UM9.2 (D); no longer UE5.1 (~{Mr}), UJ10.1 (I3)
- net M14.9: now also UM14.9 (O0b)
- net MCA6: now also P8.11 (Pin_11)
- net P4.7: now also P4.7 (Pin_7)
- net P7.9: now also R7.9 (R8); no longer R7.10 (R9)
- net PA11: now also P10.1 (Pin_1)
- net PA13: now also P10.3 (Pin_3)
- net VCC: now also P4.8 (Pin_8), P4.9 (Pin_9), P8.15 (Pin_15), P8.16 (Pin_16), UE5.1 (~{Mr}), UJ10.1 (I3), UK11.6 (E3), UL13.1 (~{R}), UL9.3 (~{RE}), UM9.10 (~{S}), UM9.12 (D)
- net ~{INTR}: now also R16.6 (R5)
- net ~{LOAD.SAR}: now also UJ7.1 (~{RE})
- net ~{PA14}: now also UA9.12 (BUS2)
- net ~{RESET2}: now also UM9.1 (~{R})
- net TIMER.Q: now reaches UF13.15 (Q5), UH13.1
- net TIMER.Q: now also UM7.8 (I3a)
- net P7.14: now reaches R11.2, UE3.18 (CE3), UF3.18 (CE3), UH3.18 (CE3), UJ3.18 (CE3), UK3.18 (CE3), UL3.18 (CE3), UM3.18 (CE3)
- net P7.14: now also P7.14 (Pin_14)
- net ~{CPU.CLKC}: now reaches UM12.9 (C)
- net DIP.O: now reaches P3.4 (Pin_4)
- net ~{PROME}: now reaches UB13.16 (E2)
- net ~{PROME}: now also UM13.7 (Q3)
- net A14.1 renamed BUS.READY
- net DBP renamed DBPO
- net E10.12 renamed END.R/~{W}
- net E8.1 renamed CYCLE.ABORT
- net E8.13 renamed BUS.END
- net TIMER: no longer names the net of UF14.9, UM9.9 (Q)
- net WAR.OVR renamed WAR.TC
- net XX.CLK renamed CPU.CLK
- net ~{E7.O1} renamed ~{BUS.ABT}
- net ~{PHI1}' renamed ~{PHI1A}
- net ~{XX.CLK}' renamed ~{CPU.CLKB}
- net ~{XX.CLK}'' renamed ~{CPU.CLKA}
- net ~{XX.CLK}''' renamed ~{CPU.CLK}
- new net P7.13: P7.13 (Pin_13), UL10.2 (D), UL10.9 (Q), UL11.13 (I1d), UM10.12
- no-connect marks 108 -> 120
Other:
- note added: "ALU"
- note added: "Address Decoding"
- note added: "Address Registers"
- note added: "CPU Primary Clock"
- note added: "CPU State Control"
- note added: "Condition Codes"
- note added: "Instruction Decoder"
- note added: "Microcode Decoders"
- note added: "Microcode ROM and Pipeline Register"
- note added: "Microcode conditionals"
- note added: "Page File"
- note added: "Pulled Up"
- note added: "Pulled up"
- note added: "Register File"
- note added: "Sequencer"
- note added: "Swapper"
- note added: "Unused"
- moved on the sheet: P4, P7, R1, R14, R17, R2, R3, R6, R8, R9, UA15E, UA15F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
