File: kicad/CPU6/CPU6.kicad_sch (KiCad schematic)
At the start: 207 parts, among them P1 Edge Connector, P10 Conn_02x08_Counter_Clockwise, P2 Connector, P3 Connector, P4 Conn_02x08_Counter_Clockwise, P5 Conn_02x25_Odd_Even, P6 Conn_02x25_Odd_Even, P7 Conn_02x07_Counter_Clockwise, P8 Conn_02x08_Counter_Clockwise

Commit message: Corrections from CPU5 reverse engineering
Parts:
- added JE3, JF3, JH3, JJ3, JK3, JL3, JM3: Conn_01x12, Connector_PinSocket_2.54mm:PinSocket_1x12_P2.54mm_Vertical, symbol Connector_Generic:Conn_01x12
- C1, C10, C11, C12, C13, C14, C15, C16, C17, C18, C19, C2, C20, C21, C22, C23, C24, C25, C26, C27, C28, C29, C3, C30, C31, C32, C33, C34, C35, C36, C37, C38, C4, C40, C41, C42, C43, C44, C45, C46, C47, C48, C49, C5, C50, C51, C6, C7, C8, C9: footprint Capacitor_THT:C_Disc_D3.0mm_W1.6mm_P2.50mm -> Capacitor_THT:C_Disc_D3.8mm_W2.6mm_P2.50mm
- C39: footprint Capacitor_THT:CP_Axial_L25.0mm_D10.0mm_P30.00mm_Horizontal -> Capacitor_THT:CP_Axial_L18.0mm_D6.5mm_P25.00mm_Horizontal
- C52, C53: footprint Capacitor_THT:CP_Axial_L34.5mm_D20.0mm_P41.00mm_Horizontal -> Capacitor_THT:CP_Axial_L29.0mm_D10.0mm_P35.00mm_Horizontal
- CR1: footprint Diode_THT:D_DO-201AD_P15.24mm_Horizontal -> Diode_THT:D_DO-35_SOD27_P10.16mm_Horizontal
- P1: footprint Connector_PinHeader_2.54mm:PinHeader_2x36_P2.54mm_Vertical -> Custom:Centurion_card_edge
- P10, P4, P8: footprint Connector_PinSocket_2.54mm:PinSocket_2x08_P2.54mm_Horizontal -> Connector_PinSocket_2.54mm:PinSocket_2x08_P2.54mm_Vertical
- P7: footprint Connector_PinSocket_2.54mm:PinSocket_2x07_P2.54mm_Horizontal -> Connector_PinSocket_2.54mm:PinSocket_2x07_P2.54mm_Vertical
- R1, R10, R11, R12, R13, R14, R15, R17, R18, R19, R2, R3, R5, R6, R8, R9: footprint Resistor_THT:R_Axial_DIN0309_L9.0mm_D3.2mm_P12.70mm_Horizontal -> Resistor_THT:R_Axial_DIN0207_L6.3mm_D2.5mm_P10.16mm_Horizontal
Connections:
- net CC.F.Q is gone; now on net CC.F: UJ11.13 (I6), UJ11.2 (I2), UM12.7 (Q2), UM14.6 (I2a), UM15.6 (I2a)
- net CC.L.Q is gone; now on net CC.L: UJ10.4 (I0), UK10.10, UK10.9, UK13.6 (I0a), UM12.10 (Q3), UM14.8 (I3a), UM15.8 (I3a)
- net CC.M.Q is gone; now on net CC.M: UJ12.6 (I0a), UM12.5 (Q1), UM14.4 (I1a), UM15.4 (I1a)
- net CC.V.Q is gone; now on net CC.V: UJ12.10 (I0b), UM12.2 (Q0), UM14.2 (I0a), UM15.2 (I0a)
- net DMA.RD is gone; now on net DMA.EN: UE11.13, UF11.12 (Q7), UM8.17 (I3b)
- net 60Hz: now also R4.4 (R3); no longer R4.7 (R6)
- net CC.F: no longer UJ11.5 (Z), UM12.6 (D2)
- net CC.L: no longer UJ10.5 (Z), UM12.11 (D3)
- net CC.M: no longer UJ12.7 (Za), UM12.4 (D1)
- net CC.V: no longer UJ12.9 (Zb), UM12.3 (D0)
- net DIP.2: now also R4.8 (R7); no longer R4.3 (R2)
- net DMA.EN: no longer UB15.10 (~{S}), UD6.1 (S), UF11.9 (Q4), UM8.11 (I0b)
- net DP4: now also UM6.18 (O0a); no longer UM6.12 (O3a)
- net DP5: now also UM6.16 (O1a); no longer UM6.14 (O2a)
- net DP6: now also UM6.14 (O2a); no longer UM6.16 (O1a)
- net DP7: now also UM6.12 (O3a); no longer UM6.18 (O0a)
- net FP.DELAY: now also R4.9 (R8); no longer R4.2 (R1)
- net GND: now also JE3.12 (Pin_12), JF3.12 (Pin_12), JH3.12 (Pin_12), JJ3.12 (Pin_12), JK3.12 (Pin_12), JL3.12 (Pin_12), JM3.12 (Pin_12)
- net MC0: now also P5.39 (Pin_39), JE3.9 (Pin_9); no longer P6.2 (Pin_2)
- net MC1: now also P5.41 (Pin_41), JE3.10 (Pin_10); no longer P6.1 (Pin_1)
- net MC10: now also P6.50 (Pin_50), JJ3.11 (Pin_11); no longer P6.19 (Pin_19)
- net MC11: now also P6.48 (Pin_48); no longer P6.21 (Pin_21)
- net MC12: now also P5.2 (Pin_2); no longer P6.23 (Pin_23)
- net MC13: now also P5.1 (Pin_1); no longer P6.25 (Pin_25)
- net MC14: now also P5.3 (Pin_3); no longer P6.27 (Pin_27)
- net MC15: now also P5.5 (Pin_5); no longer P6.29 (Pin_29)
- net MC16: now also P6.2 (Pin_2), JM3.9 (Pin_9); no longer P6.31 (Pin_31)
- net MC17: now also P6.1 (Pin_1), JM3.10 (Pin_10); no longer P6.33 (Pin_33)
- net MC18: now also P6.3 (Pin_3), JM3.11 (Pin_11); no longer P6.35 (Pin_35)
- net MC19: now also P6.5 (Pin_5); no longer P6.37 (Pin_37)
- net MC2: now also P5.43 (Pin_43), JE3.11 (Pin_11); no longer P6.3 (Pin_3)
- net MC20: now also P6.7 (Pin_7); no longer P6.39 (Pin_39)
- net MC21: now also P6.9 (Pin_9); no longer P6.41 (Pin_41)
- net MC22: now also P6.11 (Pin_11); no longer P6.43 (Pin_43)
- net MC23: now also P6.13 (Pin_13); no longer P6.45 (Pin_45)
- net MC24: now also P6.15 (Pin_15), JL3.9 (Pin_9); no longer P6.47 (Pin_47)
- net MC25: now also P6.17 (Pin_17), JL3.10 (Pin_10); no longer P6.49 (Pin_49)
- net MC26: now also P6.19 (Pin_19), JL3.11 (Pin_11); no longer P6.50 (Pin_50)
- net MC27: now also P6.21 (Pin_21); no longer P6.48 (Pin_48)
- net MC28: now also P6.23 (Pin_23); no longer P5.2 (Pin_2)
- net MC29: now also P6.25 (Pin_25); no longer P5.1 (Pin_1)
- net MC3: now also P5.45 (Pin_45); no longer P6.5 (Pin_5)
- net MC30: now also P6.27 (Pin_27); no longer P5.3 (Pin_3)
- net MC31: now also P6.29 (Pin_29); no longer P5.5 (Pin_5)
- net MC32: now also JH3.9 (Pin_9)
- net MC33: now also JH3.10 (Pin_10)
- net MC34: now also JH3.11 (Pin_11)
- net MC4: now also P5.47 (Pin_47); no longer P6.7 (Pin_7)
- net MC40: now also JF3.9 (Pin_9)
- net MC41: now also JF3.10 (Pin_10)
- net MC42: now also JF3.11 (Pin_11)
- net MC48: now also P6.31 (Pin_31), JK3.9 (Pin_9); no longer P5.39 (Pin_39)
- net MC49: now also P6.33 (Pin_33), JK3.10 (Pin_10); no longer P5.41 (Pin_41)
- net MC5: now also P5.49 (Pin_49); no longer P6.9 (Pin_9)
- net MC50: now also P6.35 (Pin_35), JK3.11 (Pin_11); no longer P5.43 (Pin_43)
- net MC51: now also P6.37 (Pin_37); no longer P5.45 (Pin_45)
- net MC52: now also P6.39 (Pin_39); no longer P5.47 (Pin_47)
- net MC53: now also P6.41 (Pin_41); no longer P5.49 (Pin_49)
- net MC54: now also P6.43 (Pin_43); no longer P5.50 (Pin_50)
- net MC55: now also P6.45 (Pin_45); no longer P5.48 (Pin_48)
- net MC6: now also P5.50 (Pin_50); no longer P6.11 (Pin_11)
- net MC7: now also P5.48 (Pin_48); no longer P6.13 (Pin_13)
- net MC8: now also P6.47 (Pin_47), JJ3.9 (Pin_9); no longer P6.15 (Pin_15)
- net MC9: now also P6.49 (Pin_49), JJ3.10 (Pin_10); no longer P6.17 (Pin_17)
- net MCA0: now also JE3.8 (Pin_8), JF3.8 (Pin_8), JH3.8 (Pin_8), JJ3.8 (Pin_8), JK3.8 (Pin_8), JL3.8 (Pin_8), JM3.8 (Pin_8)
- net MCA1: now also JE3.7 (Pin_7), JF3.7 (Pin_7), JH3.7 (Pin_7), JJ3.7 (Pin_7), JK3.7 (Pin_7), JL3.7 (Pin_7), JM3.7 (Pin_7)
- net MCA2: now also JE3.6 (Pin_6), JF3.6 (Pin_6), JH3.6 (Pin_6), JJ3.6 (Pin_6), JK3.6 (Pin_6), JL3.6 (Pin_6), JM3.6 (Pin_6)
- net MCA3: now also JE3.5 (Pin_5), JF3.5 (Pin_5), JH3.5 (Pin_5), JJ3.5 (Pin_5), JK3.5 (Pin_5), JL3.5 (Pin_5), JM3.5 (Pin_5)
- net MCA4: now also JE3.4 (Pin_4), JF3.4 (Pin_4), JH3.4 (Pin_4), JJ3.4 (Pin_4), JK3.4 (Pin_4), JL3.4 (Pin_4), JM3.4 (Pin_4)
- net MCA5: now also JE3.3 (Pin_3), JF3.3 (Pin_3), JH3.3 (Pin_3), JJ3.3 (Pin_3), JK3.3 (Pin_3), JL3.3 (Pin_3), JM3.3 (Pin_3)
- net MCA6: now also JE3.2 (Pin_2), JF3.2 (Pin_2), JH3.2 (Pin_2), JJ3.2 (Pin_2), JK3.2 (Pin_2), JL3.2 (Pin_2), JM3.2 (Pin_2)
- net MCA7: now also JE3.1 (Pin_1), JF3.1 (Pin_1), JH3.1 (Pin_1), JJ3.1 (Pin_1), JK3.1 (Pin_1), JL3.1 (Pin_1), JM3.1 (Pin_1)
- net PA12: no longer UC8.11
- net PA17: now also UC8.11
- net R/F: now also R4.7 (R6); no longer R4.4 (R3)
- net VCC: now also UD2.13 (A1), UD2.14 (A0), UD2.15 (E), UE12.11, UE12.13, UE12.5, UE12.9, UE8.8, UE8.9, UH14.12 (I5), UH14.14 (I6), UH14.15 (OEb), UJ6.3, UL13.11 (~{S}), UL13.12 (C), UL13.13 (~{K}), UL13.14 (J), UL13.15 (~{R}), UL14.1, UL14.10, UL14.2, UL14.9
- net ~{A12}: now also P1.a10 (Pin_a10); no longer P1.a9 (Pin_a9)
- net ~{A14}: now also P1.a9 (Pin_a9); no longer P1.a10 (Pin_a10)
- net ~{BUS.WAIT}: now also UE11.11, UE14.9
- net ~{DRDY}: now also R16.2 (R1); no longer R16.9 (R8)
- net ~{INC.MAR}: now also UD6.5 (I0b); no longer UD6.14 (I0d)
- net ~{INC.WAR}: now also UD6.14 (I0d); no longer UD6.5 (I0b)
- net ~{INR0}: now also R16.6 (R5); no longer R16.5 (R4)
- net ~{INR1}: now also R16.7 (R6); no longer R16.4 (R3)
- net ~{INR2}: now also R16.8 (R7); no longer R16.3 (R2)
- net ~{INR3}: now also R16.9 (R8); no longer R16.2 (R1)
- net ~{INTR}: now also R16.5 (R4); no longer R16.6 (R5)
- net ~{PE}: now also R16.3 (R2); no longer R16.8 (R7)
- net ALU.RAM3 renamed ALU.RAM7
- net B12.11 renamed REG/RDONLY
- net B15.9 renamed ~{DMA.PE}
- net BUS.END: no longer names the net of UB12.5, UE8.13
- net BUS.END: no longer UE11.11, UE14.9
- net CYCLE.ABORT: no longer names the net of UE14.13, UE8.1
- net DMA10 renamed ~{DMA.START}
- net ~{DMA.START}: now also R4.3 (R2); no longer R4.8 (R7)
- net DMA11 renamed DMA.WRITE
- net DMA.WRITE: now also R4.2 (R1); no longer R4.9 (R8)
- net DMA12 renamed ~{DMA.INTR}
- net ~{DMA.INTR}: now also R4.5 (R4); no longer R4.6 (R5)
- net DMA13 renamed ~{DMA.REQ}
- net ~{DMA.REQ}: now also R4.6 (R5); no longer R4.5 (R4)
- net DMA13.Q renamed ~{DMA.REQ.Q}
- net DMA2 renamed ~{DMA.ACT}
- net DMA5 renamed ~{DMA.END}
- net DMA6 renamed ~{DMA.EN}
- net DMA8 renamed ~{DMA.RDRDY}
- net DMA9 renamed ~{DMA.WTRDY}
- net E10.6 renamed DMAE
- net E10.6.Q renamed DMAE.Q
- net E11.6 renamed ~{DMA.RD}
- net E14.10 renamed DMA.RDY
- net INC.DMA renamed ~{INC.DMA}
- net INTR.Q renamed ~{INTR.Q}
- net L13.7 renamed DMA.END
- net LVL15.Q renamed ~{DMA.INT.Q}
- net M14.9 renamed DMA.INTR
- net M8.12 renamed DMA.START
- net M8.14 renamed DMA.READ
- net M9.5 renamed DMA.RDRDY
- net PA18 renamed RDONLY
- net TIMER.Q renamed ~{TIMER.Q}
- net X.CLK renamed DMA.CLK
- net ~{K11.O1} renamed ~{DMA.RESET}
- net ~{LVL15} renamed ~{DMA.INT}
- net ~{PA18} renamed ~{BRDONLY}
- net ~{BRDONLY}: no longer R16.7 (R6)
- net ~{PA18}' renamed ~{RDONLY}
- new net: UJ10.5 (Z), UM12.11 (D3)
- new net: UJ12.9 (Zb), UM12.3 (D0)
- new net: UJ12.7 (Za), UM12.4 (D1)
- new net: UJ11.5 (Z), UM12.6 (D2)
- new net DMA.ACT: UB15.10 (~{S}), UD6.1 (S), UF11.9 (Q4), UM8.11 (I0b)
- no-connect marks 120 -> 102
Other:
- note added: "(DMA.EN and INC.DMA) or BUS.WAIT"
- note added: "(DMA.READ and NOT.MEM) or (REG/RDONLY and DMA.WRITE) or DMA.PE"
- note added: "INC.DMA and DMA.EN"
- note added: "Interrupts"
- note added: "Parity Error"
- note added: "not (INC.DMA and DMA.EN and WAR.TC)"
- note added: "not DMA.EN or not INC.DMA"
- company: (none) -> SJSoftware
- moved on the sheet: C39, CR1, DSW1, P1, P10, P2, P3, P4, P5, P6, P7, P8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
